File: Hardware/Burocket_hardware.kicad_sch (KiCad schematic)
At the start: 0 parts

Commit message: Edited schematics
Other:
- company: (none) -> Burocket
- title: (none) -> Dumenden aviyonik pc
Changed lines of the file:
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@@
 	(generator_version "10.0")
 	(paper "A4")
+	(title_block
+		(title "Dumenden aviyonik pc")
+		(date "2026-07-08")
+		(rev "0.1")
+		(company "Burocket")
+	)
 	(sheet
 		(at 109.22 71.12)
