File: Hardware/Burocket_hardware.kicad_sch (KiCad schematic)
At the start: 0 parts

Commit message: Changed footprints, generated BOM
Other:
- note added: "BuRocket Flight Controller"
- note added: "JLCPCB Stack-up"
Changed lines of the file:
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@@
 		(company "Burocket")
 	)
+	(text "BuRocket Flight Controller"
+		(exclude_from_sim no)
+		(at 68.58 20.32 0)
+		(effects
+			(font
+				(size 7.62 7.62)
+				(thickness 1.524)
+				(bold yes)
+			)
+			(justify left)
+		)
+	)
+	(text "JLCPCB Stack-up"
+		(exclude_from_sim no)
+		(at 51.054 130.302 0)
+		(effects
+			(font
+				(size 3.81 3.81)
+				(thickness 0.4763)
+			)
+			(justify left)
+		)
+	)
 	(text "TODO:\n- Must change nmos driving E-match\n- Consider Passive components\n\n- Consider and thoroughly check all footprints\n"
 		(exclude_from_sim no)
-		(at -211.582 50.038 0)
+		(at -204.216 54.102 0)
 		(effects
 			(font
@@
 	(text "Note:\n- Buzzer simulation don't \nreally match \n"
 		(exclude_from_sim no)
-		(at -117.856 184.912 0)
+		(at -203.454 92.456 0)
 		(effects
 			(font
@@
 	)
 	(image
-		(at 68.58 29.464)
+		(at 80.772 155.702)
 		(data "iVBORw0KGgoAAAANSUhEUgAABS8AAAGVCAIAAACQNJMeAAAAA3NCSVQICAjb4U/gAAAgAElEQVR4"
 			"nOy9d5ReV3X3/937nFueMk29WcWyLMlyB/cmdxvTbCBAQioQfpSEFjpxwkt934DDSzckgEMAN2zj"
@@
 		)
 	)
+	(rule_area
+		(exclude_from_sim no)
+		(in_bom yes)
+		(on_board yes)
+		(dnp no)
+		(polyline
+			(pts
+				(xy 20.828 124.714) (xy 20.828 174.498) (xy 140.208 174.498) (xy 140.208 124.714)
+			)
+			(stroke
+				(width 0)
+				(type dash)
+			)
+			(fill
+				(type none)
+			)
+		)
+	)
 	(sheet
-		(at 131.572 77.978)
+		(at 130.302 47.244)
 		(size 18.288 14.478)
 		(exclude_from_sim no)
@@
 		)
 		(property "Sheetname" "Connections_relays"
-			(at 131.572 77.2664 0)
+			(at 130.302 46.5324 0)
 			(show_name no)
 			(do_not_autoplace no)
@@
 		)
 		(property "Sheetfile" "Connections_relays.kicad_sch"
-			(at 131.572 93.0406 0)
+			(at 130.302 62.3066 0)
 			(show_name no)
 			(do_not_autoplace no)
@@
 	)
 	(sheet
-		(at 132.588 101.854)
+		(at 131.318 71.12)
 		(size 19.05 13.335)
 		(exclude_from_sim no)
@@
 		)
 		(property "Sheetname" "Sensors"
-			(at 132.588 101.1424 0)
+			(at 131.318 70.4084 0)
 			(show_name no)
 			(do_not_autoplace no)
@@
 		)
 		(property "Sheetfile" "Sensors.kicad_sch"
-			(at 132.588 115.7736 0)
+			(at 131.318 85.0396 0)
 			(show_name no)
 			(do_not_autoplace no)
@@
 	)
 	(sheet
-		(at 107.696 101.854)
+		(at 106.426 71.12)
 		(size 19.05 13.335)
 		(exclude_from_sim no)
@@
 		)
 		(property "Sheetname" "Power"
-			(at 107.696 101.1424 0)
+			(at 106.426 70.4084 0)
 			(show_name no)
 			(do_not_autoplace no)
@@
 		)
 		(property "Sheetfile" "Power.kicad_sch"
-			(at 107.696 115.7736 0)
+			(at 106.426 85.0396 0)
 			(show_name no)
 			(do_not_autoplace no)
@@
 	)
 	(sheet
-		(at 108.204 76.962)
+		(at 106.934 46.228)
 		(size 20.066 16.002)
 		(exclude_from_sim no)
@@
 		)
 		(property "Sheetname" "MCU"
-			(at 108.204 76.2504 0)
+			(at 106.934 45.5164 0)
 			(show_name no)
 			(do_not_autoplace no)
@@
 		)
 		(property "Sheetfile" "MCU.kicad_sch"
-			(at 108.204 93.5486 0)
+			(at 106.934 62.8146 0)
 			(show_name no)
 			(do_not_autoplace no)
@@
 	)
 	(sheet
-		(at 155.448 101.727)
+		(at 154.178 70.993)
 		(size 17.78 13.335)
 		(exclude_from_sim no)
@@
 		)
 		(property "Sheetname" "LoRa"
-			(at 155.448 101.0154 0)
+			(at 154.178 70.2814 0)
 			(show_name no)
 			(do_not_autoplace no)
@@
 		)
 		(property "Sheetfile" "LoRa.kicad_sch"
-			(at 155.448 115.6466 0)
+			(at 154.178 84.9126 0)
 			(show_name no)
 			(do_not_autoplace no)
@@
 	)
 	(sheet
-		(at 155.702 77.724)
+		(at 154.432 46.99)
 		(size 19.558 13.462)
 		(exclude_from_sim no)
@@
 		)
 		(property "Sheetname" "USB-c"
-			(at 155.702 77.0124 0)
+			(at 154.432 46.2784 0)
 			(show_name no)
 			(do_not_autoplace no)
@@
 		)
 		(property "Sheetfile" "USB-c.kicad_sch"
-			(at 155.702 91.7706 0)
+			(at 154.432 61.0366 0)
 			(show_name no)
 			(do_not_autoplace no)
