File: Hardware/Power.kicad_sch (KiCad schematic)
At the start: 0 parts

Commit message: Edited schematics
Parts:
- added BT1: Battery, Connector_AMASS:AMASS_XT60-F_1x02_P7.20mm_Vertical, symbol Device:Battery
Connections:
- new net +BATT: BT1.1 (+)
- new net GND: BT1.2 (-)
Other:
- company: (none) -> Burocket
- title: (none) -> Power

Commit message: Selected components and added their properties, started the power schematics
Parts:
- added C19, C20, C25, C26, C9: C, symbol Device:C
- added C23: 100nF, Capacitor_SMD:C_0402_1005Metric, symbol Device:C
- added C24: 0.1nF, Capacitor_SMD:C_0402_1005Metric, symbol Device:C
- added L1: 9.1uH, Inductor_SMD_Wurth:L_Wurth_WE-PDF-1045, symbol Device:L
- added R21: 100k, Resistor_SMD:R_0402_1005Metric, symbol Device:R
- added R22: 13.7K, Resistor_SMD:R_0402_1005Metric, symbol Device:R
- added R23: 412k, Resistor_SMD:R_0402_1005Metric, symbol Device:R
- added R24: 97.6K, Resistor_SMD:R_0402_1005Metric, symbol Device:R
- added U2: TPS54302, TPS54302DDCR:SOT95P280X110-6N, symbol TPS54302DDCR:TPS54302DDCR
- added U8: TPS2121RUXR, footprints.ugly:RUX0012A, symbol 2026-06-29_10-29-30:TPS2121RUXR
Connections:
- net +BATT: now also C19.1, C20.1, C9.1, R23.1, U2.3 (VIN)
- net GND: now also C19.2, C20.2, C25.2, C26.2, C9.2, R22.2, R24.2, U2.1 (GND)
- new net: C24.2, R21.2, R22.1, U2.4 (FB)
- new net: C23.1, U2.6 (BOOT)
- new net: C23.2, C24.1, L1.1, U2.2 (SW)
- new net: R23.2, R24.1, U2.5 (EN)
- new net: U8.1 (OUT), U8.8 (OUT)
- new net +5V: C25.1, C26.1, L1.2, R21.1
- new net VBUS: U8.2 (IN2)
Other:
- note added: "2S BAT 6-8.4V"
- note added: "TODO: Select input and output caps"
- note added: "UVLO = 6V"
- moved on the sheet: BT1

Commit message: Added a simulations file, added App Notes file, Finalized SD-card design type shit
Connections:
- net +5V: now also U8.7 (IN1)
- net GND: now also U8.12 (GND)
Other:
- moved on the sheet: BT1, C19, C20, C23, C24, C25, C26, C9, L1, R21, R22, R23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

Commit message: +1000 Aura
Parts:
- removed C9: C, symbol Device:C
- added C35: 2.2uF, Capacitor_SMD:C_0402_1005Metric, symbol Device:C
- added C36: 10uF, Capacitor_SMD:C_0603_1608Metric, symbol Device:C
- added R29, R30, R31: 48.7K, Resistor_SMD:R_0402_1005Metric, symbol Device:R
- added R32: 28k, Resistor_SMD:R_0402_1005Metric, symbol Device:R
- added R36, R37, R38: 10k, Resistor_SMD:R_0603_1608Metric, symbol Device:R
- C19, C20: value C -> 10uF; footprint (none) -> Capacitor_SMD:C_0603_1608Metric; Distributer Link (none) -> https://www.ozdisan.com/p/smt-smd-ve-mlcc-kapasitorler-184/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; Part Number (none) -> GRT188C81C106ME13D
Connections:
- net +5V: now also R29.1, R32.1
- net +BATT: now also C36.1
- net GND: now also U8.3 (CP2), U8.9 (ST), C35.2, C36.2, R31.2, R36.2, R37.2, R38.2
- net VBUS: now also R30.1
- net +5VP: now reaches U8.1 (OUT), U8.8 (OUT)
- net at U8.10 (ILM): now also R31.1
- net at U8.11 (SS): now also C35.1
- net at U8.4 (OV2): now also R30.2, R38.1
- net at U8.5 (OV1): now also R29.2, R37.1
- net at U8.6 (PR1): now also R32.2, R36.1
Other:
- note added: "- Priority voltage: 3.77V - 4.23V considering resistor tolerance (%1) and IC accuracy tolerance (%5) - Overvoltage 1,2: 6.01V - 6.42V considering resistor tolerance (%1) and IC accuracy tolerance (%5) - Current limiting: 65.2/48.7^0.861 = 2.3A"
- note added: "ADD ESD protection to Input"
- moved on the sheet: BT1, C23, C24, C25, C26, L1, R21, R22, R23, R24, U2

Commit message: Only SSR and ferrite bead selection is left
Parts:
- removed C19, C20, C36: 10uF, Capacitor_SMD:C_0603_1608Metric, symbol Device:C
- removed C26: C, symbol Device:C
- added C38, C41, C42, C43, C44: 22uF, Capacitor_SMD:C_0805_2012Metric, symbol Device:C
- added C40: 100nF, Capacitor_SMD:C_0402_1005Metric, symbol Device:C
- added FB2, FB3: FerriteBead, symbol Device:FerriteBead
- added U3: LD1086DT33TR, Package_TO_SOT_SMD:TO-252-2, symbol Regulator_Linear:LD1086DT33TR
- BT1: Distributer Link (none) -> https://www.robo90.com/xt60-konnektor-lipo-pil-konnektoru-d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; Part Number (none) -> XT60
- C25: value C -> 47uF; footprint (none) -> Capacitor_SMD:C_1210_3225Metric; Distributer Link (none) -> https://www.ozdisan.com/p/smt-smd-ve-mlcc-kapasitorler-184/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; Part Number (none) -> CL32A476KOJNNNE
- R36, R37, R38: footprint Resistor_SMD:R_0603_1608Metric -> Resistor_SMD:R_0402_1005Metric; Distributer Link https://www.ozdisan.com/p/smt-smd-ve-cip-direncler-194/pana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 -> https://www.ozdisan.com/p/smt-smd-ve-cip-direncler-194/roya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; Part Number ERJ3EKF1002V -> CQ02WGF1002TCE
Connections:
- net +5V: now also FB2.1; no longer C25.1, L1.2, R21.1
- net +5VP: now also C38.1, U3.3 (IN)
- net +BATT: now also C42.1, C43.1, C44.1
- net GND: now also C38.2, C40.1, C41.2, C42.2, C43.2, C44.2, U3.1 (ADJ/GND)
- net at C24.1, L1.1, U2.2 (SW): no longer C23.2
- new net: C25.1, FB2.2, L1.2, R21.1
- new net: C41.1, FB3.2, U3.2 (OUT)
- new net +3.3V: C40.2, FB3.1
Other:
- note added: "- MCU - Micro SD-card"
- note added: "- Priority voltage: 3.77V - 4.23V considering resistor tolerance (%1) and IC accuracy tolerance (%5) - Overvoltage 1,2: 6.01V - 6.42V considering resistor tolerance (%1) and IC accuracy tolerance (%5) - Current limiting: 65.2/48.7^0.861 = 2.3A (possibly change)"
- note added: "2S 6-8.4V"
- note added: "Add heatsink above the LDO, thermal vias, copper pad underneath"
- note added: "Buck Converter"
- note added: "Buck converter ----->"
- note added: "Current ≈400mA"
- note added: "MAX Current ≈260mA"
- note added: "MAX Current ≈660mA"
- note added: "OR"
- note added: "Sensors: - IMU & Gyro - GPS - IMU - BARO"
- note added: "TODO: - Select input and output caps - Add ferrite bead"
- note added: "Total Power dissipation = 0.663A X (5.0V - 3.3V) = 1.127W which is, pretty insane"
- note removed: "- Priority voltage: 3.77V - 4.23V considering resistor tolerance (%1) and IC accuracy tolerance (%5) - Overvoltage 1,2: 6.01V - 6.42V considering resistor tolerance (%1) and IC accuracy tolerance (%5) - Current limiting: 65.2/48.7^0.861 = 2.3A"
- note removed: "---->"
- note removed: "TODO: Select input and output caps"
- moved on the sheet: BT1, C23, C24, C25, C35, L1, R21, R22, R23, R24, R29, R30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

Commit message: Ne yazacagimi bilemedim
Other:
- note removed: "ADD ESD protection to Input"
- note removed: "TODO: - Select input and output caps - Add ferrite bead"
Changed lines of the file:
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@@
-		)
-	)
-	(text "ADD ESD protection to Input"
-		(exclude_from_sim no)
-		(at 17.145 -20.955 0)
-		(effects
-			(font
-				(size 5.08 5.08)
-				(thickness 1.016)
-				(bold yes)
-			)
-			(justify left)
 		)
 	)
@@
 				(bold yes)
 			)
-			(justify left)
-		)
-	)
-	(text "TODO: \n- Select input and output caps\n- Add ferrite bead"
-		(exclude_from_sim no)
-		(at -130.175 23.495 0)
-		(effects
-			(font
-				(size 5.08 5.08)
-				(thickness 1.016)
-				(bold yes)
-			)

Commit message: Updated schematics
Connections:
- net at C23.2: now also C24.1, L1.1, U2.2 (SW)
Other:
- note added: "Do calculations"
Changed lines of the file:
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@@
 		)
 	)
-	(text "Buck converter"
-		(exclude_from_sim no)
-		(at 50.165 34.925 0)
+	(text "Do calculations"
+		(exclude_from_sim no)
+		(at 51.308 49.784 0)
 		(effects
 			(font
@@
 		)
 	)
+	(text "Buck converter"
+		(exclude_from_sim no)
+		(at 50.165 34.925 0)
+		(effects
+			(font
+				(size 2.54 2.54)
+				(thickness 0.508)
+				(bold yes)
+			)
+			(justify left)
+		)
+	)
 	(text "LDO"
 		(exclude_from_sim no)
@@
 	)
 	(junction
+		(at 120.65 60.325)
+		(diameter 0)
+		(color 0 0 0 0)
+	)
+	(junction
 		(at 127.762 78.74)
 		(diameter 0)
@@
 	(wire
 		(pts
-			(xy 120.65 60.452) (xy 120.65 62.738)
+			(xy 120.65 60.198) (xy 120.65 60.325)
 		)
 		(stroke
@@
 	(wire
 		(pts
-			(xy 120.65 62.738) (xy 119.126 62.738)
+			(xy 120.65 62.484) (xy 119.126 62.484)
 		)
 		(stroke
@@
 	(wire
 		(pts
-			(xy 119.126 62.738) (xy 119.126 67.818)
+			(xy 119.126 62.484) (xy 119.126 67.818)
 		)
 		(stroke
@@
 		)
 		(stroke
+			(width 0)
+			(type default)
+		)
+	)
+	(wire
+		(pts
+			(xy 120.65 60.325) (xy 120.65 62.484)
+		)
+		(stroke

Commit message: Commit bulamadim :)
Parts:
- added C30, C31: 100nF, Capacitor_SMD:C_0402_1005Metric, symbol Device:C
- added R60, R61: 4.7, Resistor_SMD:R_0402_1005Metric, symbol Device:R
- added R_Shunt1: 5m, Resistor_SMD:R_1206_3216Metric, symbol Device:R
- added U10: INA226, Package_SO:TSSOP-10_3x3mm_P0.5mm, symbol Sensor_Energy:INA226
Connections:
- net +3.3V: now also C30.1, U10.6 (VS)
- net +BATT: now also C31.1, R60.1, R_Shunt1.1, U10.8 (Vbus); no longer C42.1, C43.1, C44.1, R23.1, U2.3 (VIN)
- net GND: now also C30.2, U10.1 (A1), U10.2 (A0), U10.7 (GND)
- new net: R60.2, U10.10 (Vin+)
- new net: R61.2, U10.9 (Vin-)
- new net: C42.1, C43.1, R23.1, U2.3 (VIN)
- new net Sense_SCL: U10.4 (SDA)
- new net Sense_SDA: U10.5 (SCL)
- new net Sense_alert: U10.3 (~{Alert})
- new net shunt-: C31.2, C44.1, R61.1, R_Shunt1.2
Other:
- note added: "Current Sensing"
- moved on the sheet: BT1, C23, C24, C25, C38, C40, C41, C42, C43, C44, FB2, FB3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
