File: Hardware/Power.kicad_sch (KiCad schematic)
At the start: 34 parts, among them U10 INA226, U2 TPS54302, U3 LD1086DT33TR, U8 TPS2121RUXR

Commit message: Added New file for additional resources used, Changed LDO for lower noise, changed buck converter for higher switching speed, smaller inductance value, better transient current response
Parts:
- added C52, C54, C55: 2.2uF, Capacitor_SMD:C_0603_1608Metric, symbol Device:C
- added C53, C57: 22uF, Capacitor_SMD:C_0805_2012Metric, symbol Device:C
- added C56, C58, C59: 100nF, Capacitor_SMD:C_0402_1005Metric, symbol Device:C
- added C60, C61, C62: C, symbol Device:C
- added L2: L, symbol Device:L
- added R1, R6, R7, R8: R, symbol Device:R
- added R75: 22, Resistor_SMD:R_0402_1005Metric, symbol Device:R
- added U12: TPS7A4701, Package_DFN_QFN:Texas_RGW0020A_VQFN-20-1EP_5x5mm_P0.65mm_EP3.15x3.15mm_ThermalVias, symbol TPS2121:TPS7A8101
- added U13: TPS56339, Package_TO_SOT_SMD:SOT-23-6, symbol Regulator_Switching:TPS56339DDC
- C35: footprint Capacitor_SMD:C_0402_1005Metric -> Capacitor_SMD:C_0603_1608Metric; Distributer Link http://ozdisan.com/p/smt-smd-ve-mlcc-kapasitorler-184/murat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 -> https://www.ozdisan.com/p/smt-smd-ve-mlcc-kapasitorler-184/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; Part Number GRT155C81A225ME13D -> CL10B225KP8NNNC
Connections:
- net +3.3V: now also C52.1, C53.1, C55.1, C56.2, U12.1 (Vout), U12.20 (Vout), U12.3 (FB); no longer C40.2
- net +5V: now also C60.1, C62.1, L2.2, R7.1; no longer FB2.1
- net +5VP: now also C40.2, C57.1, C58.2, U12.13 (EN), U12.15 (Vin), U12.16 (Vin)
- net +BATT: now also C61.1, R6.1, U13.3 (VIN)
- net GND: now also C52.2, C53.2, C54.2, C55.2, C56.1, C57.2, C58.1, C61.2, R1.2, R8.2, U12.11 (0P2V), U12.12 (0P1V), U12.17 (NC), U12.18 (NC), U12.19 (NC), U12.2 (NC), U12.7 (GND), U12.8 (1P6V), U13.1 (GND)
- net shunt-: now also C42.1, C43.1, R23.1, U2.3 (VIN)
- net at C25.1, L1.2, R21.1: no longer FB2.2
- new net: C62.2, R7.2, R8.1, U13.4 (FB)
- new net: C59.1, L2.1, U13.2 (SW)
- new net: C54.1, U12.14 (NR)
- new net: R1.1, R6.2, U13.5 (EN)
- new net: R75.2, U13.6 (BOOT)
- new net: C59.2, R75.1
- no-connect marks 0 -> 5
Other:
- note added: "Calculate the following for the buck converter: - EN pin resistor values - Soft start: 5ms safety - Select components - Calculate Output voltage ripple value - delta Vin/delta Vout - FB pin resistors"
- note added: "Current LDO options: - TPS7A8101 3.62 euro"
- note removed: "Buck Converter"
- note removed: "Current ≈400mA"
- note removed: "MAX Current ≈260mA"
- note removed: "OR"
- moved on the sheet: BT1, C23, C24, C25, C30, C31, C38, C40, C41, C42, C43, C44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

Commit message: Added Impedance matching calculations, finished buck converter calculations, finalized buzzer circuitry
Parts:
- removed BT1: Battery, Connector_AMASS:AMASS_XT60-F_1x02_P7.20mm_Vertical, symbol Device:Battery
- removed C23, C40, C59: 100nF, Capacitor_SMD:C_0402_1005Metric, symbol Device:C
- removed C24: 0.1nF, Capacitor_SMD:C_0402_1005Metric, symbol Device:C
- removed C25: 47uF, Capacitor_SMD:C_1210_3225Metric, symbol Device:C
- removed C38, C41, C42, C43, C44: 22uF, Capacitor_SMD:C_0805_2012Metric, symbol Device:C
- removed C52: 2.2uF, Capacitor_SMD:C_0603_1608Metric, symbol Device:C
- removed C60, C61, C62: C, symbol Device:C
- removed FB2, FB3: FerriteBead, symbol Device:FerriteBead
- removed L1: 9.1uH, Inductor_SMD_Wurth:L_Wurth_WE-PDF-1045, symbol Device:L
- removed L2: L, symbol Device:L
- removed R1, R6, R7, R8: R, symbol Device:R
- removed R21: 100k, Resistor_SMD:R_0402_1005Metric, symbol Device:R
- removed R22: 13.7K, Resistor_SMD:R_0402_1005Metric, symbol Device:R
- removed R23: 412k, Resistor_SMD:R_0402_1005Metric, symbol Device:R
- removed R24: 97.6K, Resistor_SMD:R_0402_1005Metric, symbol Device:R
- removed R75: 22, Resistor_SMD:R_0402_1005Metric, symbol Device:R
- removed R_Shunt1: 5m, Resistor_SMD:R_1206_3216Metric, symbol Device:R
- removed U13: TPS56339, Package_TO_SOT_SMD:SOT-23-6, symbol Regulator_Switching:TPS56339DDC
- removed U2: TPS54302, TPS54302DDCR:SOT95P280X110-6N, symbol TPS54302DDCR:TPS54302DDCR
- removed U3: LD1086DT33TR, Package_TO_SOT_SMD:TO-252-2, symbol Regulator_Linear:LD1086DT33TR
- added C63, C67, C71: 100nF, Capacitor_SMD:C_0402_1005Metric, symbol Device:C
- added C64, C69, C70: 47uF, Capacitor_SMD:C_1210_3225Metric, symbol Device:C
- added C65: 0.1nF, Capacitor_SMD:C_0402_1005Metric, symbol Device:C
- added L3: 6.8uH, Inductor_SMD:L_Wuerth_XHMI-6060, symbol Device:L
- added R76: 53k6, Capacitor_SMD:C_0402_1005Metric, symbol Device:R
- added R77: 10k, Resistor_SMD:R_0402_1005Metric, symbol Device:R
- added R78: 200k, Resistor_SMD:R_0402_1005Metric, symbol Device:R
- added R79: 44.2k, Capacitor_SMD:C_0402_1005Metric, symbol Device:R
- added U14: TPS62933, Package_TO_SOT_SMD:SOT-583-8, symbol Regulator_Switching:TPS62933
Connections:
- net +5V: now also C64.1, C65.1, C69.1, L3.2, R76.1
- net +BATT: now also C70.1, C71.2, R78.1, U14.3 (VIN); no longer C31.1, R60.1
- net GND: now also C64.2, C67.2, C69.2, C70.2, C71.1, R77.2, R79.2, U14.4 (GND)
- new net: C65.2, R76.2, R77.1, U14.8 (FB)
- new net: C67.1, U14.7 (SS)
- new net: C63.1, U14.6 (BST)
- new net: C63.2, L3.1, U14.5 (SW)
- new net: R78.2, R79.1, U14.2 (EN)
- new net shunt+: C31.1, R60.1
- no-connect marks 5 -> 6
Other:
- note added: "These are theoretical values"
- note removed: "2S BAT 6-8.4V"
- note removed: "Add heatsink above the LDO, thermal vias, copper pad underneath"
- note removed: "Calculate the following for the buck converter: - EN pin resistor values - Soft start: 5ms safety - Select components - Calculate Output voltage ripple value - delta Vin/delta Vout - FB pin resistors"
- note removed: "Current LDO options: - TPS7A8101 3.62 euro"
- note removed: "Do calculations"
- note removed: "Total Power dissipation = 0.663A X (5.0V - 3.3V) = 1.127W which is, pretty insane"
- note removed: "UVLO = 6V"
- moved on the sheet: C30, C31, C53, C54, C55, C56, C57, C58, R60, R61, U10, U12

Commit message: Changed footprints, generated BOM
Parts:
- removed C63, C67, C71: 100nF, Capacitor_SMD:C_0402_1005Metric, symbol Device:C
- removed R36, R37, R38, R77: 10k, Resistor_SMD:R_0402_1005Metric, symbol Device:R
- removed R60, R61: 4.7, Resistor_SMD:R_0402_1005Metric, symbol Device:R
- added BT1: Battery, Connector_AMASS:AMASS_XT60-M_1x02_P7.20mm_Vertical, symbol Device:Battery
- added C32, C44, C59, C60: 100nF, Capacitor_SMD:C_0603_1608Metric, symbol Device:C
- added R28, R33: 4.7, Resistor_SMD:R_0603_1608Metric, symbol Device:R
- added R92, R93, R94, R95: 10k, Resistor_SMD:R_0603_1608Metric, symbol Device:R
- C30, C31, C56, C58: footprint Capacitor_SMD:C_0402_1005Metric -> Capacitor_SMD:C_0603_1608Metric; Distributer Link https://www.ozdisan.com/p/smt-smd-ve-mlcc-kapasitorler-184/murata-grt155r71e104ke01d-1074547 -> https://www.ozdisan.com/p/smt-smd-ve-mlcc-kapasitorler-184/samsung-cl10b104ko8wpnc-522227; Part Number GRT155R71E104KE01D -> CL10B104KO8WPNC
- C65: value 0.1nF -> 47pF; footprint Capacitor_SMD:C_0402_1005Metric -> Capacitor_SMD:C_0603_1608Metric; Distributer Link https://www.ozdisan.com/p/smt-smd-ve-mlcc-kapasitorler-184/murata-gcm1555c1h101ja16d-623015 -> https://www.ozdisan.com/p/smt-smd-ve-mlcc-kapasitorler-184/samsung-cl10c470jb81pnc-522565; Part Number GCM1555C1H101JA16D -> CL10C470JB81PNC
- L3: Distributer Link (none) -> https://www.mouser.com.tr/en/ProductDetail/Wurth-Elektronik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
- R29, R30, R31: footprint Resistor_SMD:R_0402_1005Metric -> Resistor_SMD:R_0603_1608Metric; Distributer Link https://www.ozdisan.com/p/smt-smd-ve-cip-direncler-194/royalohm-hp02waf4872tce-959788 -> https://www.ozdisan.com/p/smt-smd-ve-cip-direncler-194/royalohm-0603saf4872t5e-514500; Part Number HP02WAF4872TCE -> 0603SAF4872T5E
- R32: footprint Resistor_SMD:R_0402_1005Metric -> Resistor_SMD:R_0603_1608Metric; Distributer Link https://www.ozdisan.com/p/smt-smd-ve-cip-direncler-194/vish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 -> https://www.ozdisan.com/p/smt-smd-ve-cip-direncler-194/roya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; Part Number CRCW040228K0FKED -> 0603SAF2802T5E
- R78: footprint Resistor_SMD:R_0402_1005Metric -> Resistor_SMD:R_0603_1608Metric; Distributer Link https://www.ozdisan.com/p/smt-smd-ve-cip-direncler-194/yage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 -> https://www.ozdisan.com/p/smt-smd-ve-cip-direncler-194/roya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; Part Number RC0402JR-07200KL -> TC0325B2003T5C
- R79: Distributer Link https://www.ozdisan.com/p/smt-smd-ve-cip-direncler-194/yage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 -> https://www.ozdisan.com/p/smt-smd-ve-cip-direncler-194/vish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
Connections:
- net +3.3V: now also C56.1; no longer C56.2
- net +5VP: now also C58.1; no longer C58.2
- net +BATT: now also BT1.1 (+), C32.1, C44.1
- net GND: now also C56.2, C58.2, BT1.2 (-), C32.2, C44.2, C59.2, R92.2, R93.2, R94.2, R95.2; no longer C56.1, C58.1
- net shunt+: now also R28.1
- net shunt-: now also R33.1
- net at C65.2, R76.2, U14.8 (FB): now also R95.1
- net at U14.7 (SS): now also C59.1
- net at U10.10 (Vin+): now also R28.2
- net at U14.6 (BST): now also C60.1
- net at L3.1, U14.5 (SW): now also C60.2
- net at U10.9 (Vin-): now also R33.2
- net at R32.2, U8.6 (PR1): now also R92.1
- net at R30.2, U8.4 (OV2): now also R94.1
- net at R29.2, U8.5 (OV1): now also R93.1
Other:
- moved on the sheet: C53, C55, C64, C65, C69, C70, R76

Commit message: Final changes
Parts:
- added R_Shunt1: 10m, Resistor_SMD:R_1206_3216Metric, symbol Device:R
Connections:
- net shunt+ is gone; now on net +BATT: C31.1, R28.1
- net +BATT: now also R_Shunt1.1; no longer C44.1, C70.1, R78.1, U14.3 (VIN)
- net shunt-: now also C44.1, C70.1, R78.1, U14.3 (VIN), R_Shunt1.2
Changed lines of the file:
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@@
 	(wire
 		(pts
-			(xy 23.368 63.246) (xy 60.198 63.246)
+			(xy 23.368 63.246) (xy 34.798 63.246)
 		)
 		(stroke
@@
 	(wire
 		(pts
+			(xy 42.418 63.246) (xy 60.198 63.246)
+		)
+		(stroke
+			(width 0)
+			(type default)
+		)
+	)
+	(wire
+		(pts
 			(xy 207.518 50.419) (xy 207.518 53.086)
 		)
@@
 		)
 	)
+	(label "shunt-"
+		(at 42.418 63.246 0)
+		(effects
+			(font
+				(size 1.27 1.27)
+			)
+			(justify left bottom)
+		)
+	)
+	(label "shunt+"
+		(at 34.798 63.246 180)
+		(effects
+			(font
+				(size 1.27 1.27)
+			)
+			(justify right bottom)
+		)
+	)
 	(label "shunt+"
 		(at 201.168 139.192 180)
@@
 					(unit 1)
 				)
+			)
+		)
+	)
+	(symbol
+		(lib_id "Device:R")
+		(at 38.608 63.246 90)
+		(unit 1)
+		(body_style 1)
+		(exclude_from_sim no)
+		(in_bom yes)
+		(on_board yes)
+		(in_pos_files yes)
+		(dnp no)
+		(fields_autoplaced yes)
+		(property "Reference" "R_Shunt1"
+			(at 38.608 57.15 90)
+			(show_name no)
+			(do_not_autoplace no)
+			(effects
+				(font
+					(size 1.27 1.27)
+				)
+			)
+		)
+		(property "Value" "10m"
+			(at 38.608 59.69 90)
+			(show_name no)
+			(do_not_autoplace no)
+			(effects
+				(font
+					(size 1.27 1.27)
+				)
+			)
+		)
+		(property "Footprint" "Resistor_SMD:R_1206_3216Metric"
+			(at 38.608 65.024 90)
+			(hide yes)
+			(show_name no)
+			(do_not_autoplace no)
+			(effects
+				(font
+					(size 1.27 1.27)
+				)
+			)
+		)
+		(property "Datasheet" "https://cdn.ozdisan.com/public/product/assets/OHMITE_res_pcs.pdf?response-content-type=application%2Fpdf&response-content-disposition=inline"
+			(at 38.608 63.246 0)
+			(hide yes)
+			(show_name no)
+			(do_not_autoplace no)
+			(effects
+				(font
+					(size 1.27 1.27)
+				)
+			)
+		)
+		(property "Description" "RES.(3216) 1206 10m Ohms 0.5% 1W AEC-Q200"
+			(at 38.608 63.246 0)
+			(hide yes)
+			(show_name no)
+			(do_not_autoplace no)
+			(effects
+				(font
+					(size 1.27 1.27)
+				)
+			)
+		)
+		(property "Distributer Link" "https://www.ozdisan.com/p/smt-smd-ve-cip-direncler-194/ohmite-pcs1206dr0100et-955732"
+			(at 38.608 63.246 0)
+			(hide yes)
+			(show_name no)
+			(do_not_autoplace no)
+			(effects
+				(font
+					(size 1.27 1.27)
+				)
+			)
+		)
+		(property "Part Number" "PCS1206DR0100ET"
+			(at 38.608 63.246 0)
+			(hide yes)
+			(show_name no)
+			(do_not_autoplace no)
+			(effects
+				(font
+					(size 1.27 1.27)
+				)
+			)
+		)
+		(pin "2"
+		)
+		(pin "1"
+		)
+		(instances
+			(project "Burocket_hardware"
+				(path "/ece13985-822e-4117-ba82-38a772aa2f0c/4f4e3209-699f-4841-81bd-9de78787b576"
+					(reference "R_Shunt1")
+					(unit 1)
+				)

Commit message: Final touches
Parts:
- R32: Distributer Link https://www.ozdisan.com/p/smt-smd-ve-cip-direncler-194/roya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 -> https://www.mouser.com.tr/en/ProductDetail/Vishay-Beyschlag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; Part Number 0603SAF2802T5E -> MCT06030C2802FP500
- R76: footprint Capacitor_SMD:C_0402_1005Metric -> Resistor_SMD:R_0603_1608Metric; Distributer Link https://www.ozdisan.com/p/smt-smd-ve-cip-direncler-194/roya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 -> https://www.mouser.com.tr/en/ProductDetail/YAGEO/RT0603BRD0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; Part Number 0402WGF5362TCE -> RT0603BRD0753K6L
- R79: footprint Capacitor_SMD:C_0402_1005Metric -> Resistor_SMD:R_0603_1608Metric; Distributer Link https://www.ozdisan.com/p/smt-smd-ve-cip-direncler-194/vish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 -> https://www.mouser.com.tr/en/ProductDetail/YAGEO/RT0603FRE0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; Part Number RC0402FR-0744K2L -> RT0603FRE0744K2L
- R_Shunt1: value 10m -> 5m; Distributer Link https://www.ozdisan.com/p/smt-smd-ve-cip-direncler-194/ohmi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 -> http://mouser.com.tr/en/ProductDetail/Vishay-Dale/WSLP12065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; Part Number PCS1206DR0100ET -> WSLP12065L000FEA
Changed lines of the file:
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@@
 			)
 		)
-		(property "Datasheet" "https://cdn.ozdisan.com/public/product/assets/general_royalohm.pdf?response-content-type=application%2Fpdf&response-content-disposition=inline"
+		(property "Datasheet" "vishay.com/doc?28705"
 			(at 207.518 45.974 0)
 			(hide yes)
@@
 			)
 		)
-		(property "Description" "RES.(1005) 0402 28K Ohms 1% 1/16W 100PPM Automotive(AEC-Q200)"
+		(property "Description" "Thin Film Resistors - SMD MCT 0603-50 1% P5 28K"
 			(at 207.518 45.974 0)
 			(hide yes)
@@
 			)
 		)
-		(property "Distributer Link" "https://www.ozdisan.com/p/smt-smd-ve-cip-direncler-194/royalohm-0603saf2802t5e-505932"
+		(property "Distributer Link" "https://www.mouser.com.tr/en/ProductDetail/Vishay-Beyschlag/MCT06030C2802FP500?qs=hjSuqQECij8jE6Kw0BZ0wA%3D%3D"
 			(at 207.518 45.974 0)
 			(hide yes)
@@
 			)
 		)
-		(property "Part Number" "0603SAF2802T5E"
+		(property "Part Number" "MCT06030C2802FP500"
 			(at 207.518 45.974 0)
 			(hide yes)
@@
 			)
 		)
-		(property "Footprint" "Capacitor_SMD:C_0402_1005Metric"
+		(property "Footprint" "Resistor_SMD:R_0603_1608Metric"
 			(at 116.84 76.708 90)
 			(hide yes)
@@
 			)
 		)
-		(property "Datasheet" ""
+		(property "Datasheet" "https://www.mouser.com.tr/datasheet/3/72/1/PYU_RT_1_TO_0_01_ROHS_L.pdf"
 			(at 118.618 76.708 0)
 			(hide yes)
@@
 			)
 		)
-		(property "Description" "RES.(1005) 0402 53.6K Ohms 1% 1/16W 100PPM"
+		(property "Description" "Thin Film Resistors - SMD 1/10W 53.6K ohm .1% 25ppm"
 			(at 118.618 76.708 0)
 			(hide yes)
@@
 			)
 		)
-		(property "Distributer Link" "https://www.ozdisan.com/p/smt-smd-ve-cip-direncler-194/royalohm-0402wgf5362tce-506373"
+		(property "Distributer Link" "https://www.mouser.com.tr/en/ProductDetail/YAGEO/RT0603BRD0753K6L?qs=gY0y7AQI9SNAby5h%2F1y0lQ%3D%3D"
 			(at 118.618 76.708 0)
 			(hide yes)
@@
 			)
 		)
-		(property "Part Number" "0402WGF5362TCE"
+		(property "Part Number" "RT0603BRD0753K6L"
 			(at 118.618 76.708 0)
 			(hide yes)
@@
 			)
 		)
-		(property "Footprint" "Capacitor_SMD:C_0402_1005Metric"
+		(property "Footprint" "Resistor_SMD:R_0603_1608Metric"
 			(at 75.438 78.994 90)
 			(hide yes)
@@
 			)
 		)
-		(property "Datasheet" "https://cdn.ozdisan.com/public/product/assets/dcrcwe3.pdf?response-content-type=application%2Fpdf&response-content-disposition=inline"
+		(property "Datasheet" "https://www.mouser.com.tr/en/ProductDetail/YAGEO/RT0603FRE0744K2L?qs=4CyHz7GXqSgyo9YOc1MhMQ%3D%3D"
 			(at 77.216 78.994 0)
 			(hide yes)
@@
 			)
 		)
-		(property "Description" "RES.(1005) 0402 42.2K Ohms 1% 1/16W 100PPM"
+		(property "Description" "Thin Film Resistors - SMD 1/10W 44.2K ohm 1% 50ppm"
 			(at 77.216 78.994 0)
 			(hide yes)
@@
 			)
 		)
-		(property "Distributer Link" "https://www.ozdisan.com/p/smt-smd-ve-cip-direncler-194/vishay-crcw040242k2fked-516132"
+		(property "Distributer Link" "https://www.mouser.com.tr/en/ProductDetail/YAGEO/RT0603FRE0744K2L?qs=4CyHz7GXqSgyo9YOc1MhMQ%3D%3D"
 			(at 77.216 78.994 0)
 			(hide yes)
@@
 			)
 		)
-		(property "Part Number" "RC0402FR-0744K2L"
+		(property "Part Number" "RT0603FRE0744K2L"
 			(at 77.216 78.994 0)
 			(hide yes)
@@
 			)
 		)
-		(property "Value" "10m"
+		(property "Value" "5m"
 			(at 38.608 59.69 90)
 			(show_name no)
@@
 			)
 		)
-		(property "Datasheet" "https://cdn.ozdisan.com/public/product/assets/OHMITE_res_pcs.pdf?response-content-type=application%2Fpdf&response-content-disposition=inline"
+		(property "Datasheet" "https://www.mouser.com.tr/en/ProductDetail/Vishay-Dale/WSLP12065L000FEA?qs=eFWhpKjIuGhd%2FhmgEVginw%3D%3D"
 			(at 38.608 63.246 0)
 			(hide yes)
@@
 			)
 		)
-		(property "Description" "RES.(3216) 1206 10m Ohms 0.5% 1W AEC-Q200"
+		(property "Description" "Current Sense Resistors - SMD 1Watt 0.005Ohms 1%"
 			(at 38.608 63.246 0)
 			(hide yes)
@@
 			)
 		)
-		(property "Distributer Link" "https://www.ozdisan.com/p/smt-smd-ve-cip-direncler-194/ohmite-pcs1206dr0100et-955732"
+		(property "Distributer Link" "http://mouser.com.tr/en/ProductDetail/Vishay-Dale/WSLP12065L000FEA?qs=eFWhpKjIuGhd%2FhmgEVginw%3D%3D"
 			(at 38.608 63.246 0)
 			(hide yes)
@@
 			)
 		)
-		(property "Part Number" "PCS1206DR0100ET"
+		(property "Part Number" "WSLP12065L000FEA "
 			(at 38.608 63.246 0)
 			(hide yes)
