File: Hardware/LoRa.kicad_sch (KiCad schematic)
At the start: 0 parts

Commit message: Ne yazacagimi bilemedim
Changed lines of the file:
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@@
+		)
+	)
+	(global_label "RF_TX"
+		(shape output)
+		(at 56.134 98.552 180)
+		(fields_autoplaced yes)
+		(effects
+			(font
+				(size 1.27 1.27)
+			)
+			(justify right)
+		)
+		(property "Intersheetrefs" "${INTERSHEET_REFS}"
+			(at 47.6455 98.552 0)
+			(hide yes)
+			(show_name no)
+			(do_not_autoplace no)
+			(effects
+				(font
+					(size 1.27 1.27)
+				)
+				(justify right)
+			)
+		)
+	)
+	(global_label "RF_RX"
+		(shape input)
+		(at 56.134 101.346 180)
+		(fields_autoplaced yes)
+		(effects
+			(font
+				(size 1.27 1.27)
+			)
+			(justify right)
+		)
+		(property "Intersheetrefs" "${INTERSHEET_REFS}"
+			(at 47.3431 101.346 0)
+			(hide yes)
+			(show_name no)
+			(do_not_autoplace no)
+			(effects
+				(font
+					(size 1.27 1.27)
+				)
+				(justify right)
+			)
 		)
 	)

Commit message: Commit bulamadim :)
Parts:
- added C34, C49, C50: 100uF, Capacitor_Tantalum_SMD:CP_EIA-6032-20_AVX-F, symbol Device:C
- added C51: 100nF, Capacitor_SMD:C_0402_1005Metric, symbol Device:C
- added J8: Conn_01x07_Pin, symbol Connector:Conn_01x07_Pin
Connections:
- net RF_RX: now also J8.4 (Pin_4)
- net RF_TX: now also J8.3 (Pin_3)
- new net +5V: C34.1, C49.1, C50.1, C51.1, J8.6 (Pin_6)
- new net GND: C34.2, C49.2, C50.2, C51.2, J8.7 (Pin_7)
- new net RF_AUX: J8.5 (Pin_5)
- new net RF_M0: J8.1 (Pin_1)
- new net RF_M1: J8.2 (Pin_2)
Other:
- note added: "LoRa Module"
- note removed: "- Add Switches for mode selection - Add decouple capacitor bank - Add the footprint"

Commit message: Added New file for additional resources used, Changed LDO for lower noise, changed buck converter for higher switching speed, smaller inductance value, better transient current response
Parts:
- J8: footprint (none) -> footprints:E32-900T30D; now left out of the parts list
Changed lines of the file:
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@@
 		(body_style 1)
 		(exclude_from_sim no)
-		(in_bom yes)
+		(in_bom no)
 		(on_board yes)
 		(in_pos_files yes)
@@
 			)
 		)
-		(property "Footprint" ""
+		(property "Footprint" "footprints:E32-900T30D"
 			(at 178.562 98.298 0)
 			(hide yes)
@@
 			(at 178.562 98.298 0)
 			(hide yes)
+			(show_name no)
+			(do_not_autoplace no)
+			(effects
+				(font
+					(size 1.27 1.27)
+				)
+			)
+		)
+		(property "Distributer Link" ""
+			(at 178.562 98.298 0)
+			(hide yes)
+			(show_name no)
+			(do_not_autoplace no)
+			(effects
+				(font
+					(size 1.27 1.27)
+				)
+			)
+		)
+		(property "Part Number" ""
+			(at 178.562 98.298 0)
+			(hide yes)

Commit message: Added Impedance matching calculations, finished buck converter calculations, finalized buzzer circuitry
Other:
- note added: "Possibly Make PDN simulation to test voltage sag additionally to buck converter voltage sag"
- moved on the sheet: C34, C49, C50, C51, J8

Commit message: Changed footprints, generated BOM
Parts:
- C51: footprint Capacitor_SMD:C_0402_1005Metric -> Capacitor_SMD:C_0603_1608Metric; Distributer Link https://www.ozdisan.com/p/smt-smd-ve-mlcc-kapasitorler-184/murata-grt155r71e104ke01d-1074547 -> https://www.ozdisan.com/p/smt-smd-ve-mlcc-kapasitorler-184/samsung-cl10b104ko8wpnc-522227; Part Number GRT155R71E104KE01D -> CL10B104KO8WPNC
