File: Hardware/Sensors.kicad_sch (KiCad schematic)
At the start: 29 parts, among them Q7 BCR116, U5 MS5611-01BA, U6 ICM-42688-P, U7 ADXL375BCCZ-RL7, U9 MAX-M10N

Commit message: Changed footprints, generated BOM
Parts:
- removed C32: 0.1nF, Capacitor_SMD:C_0402_1005Metric, symbol Device:C
- removed C8, C9: 100nF, Capacitor_SMD:C_0402_1005Metric, symbol Device:C
- removed R54: 10k, Resistor_SMD:R_0402_1005Metric, symbol Device:R
- removed R57, R58, R59, R67: 22, Resistor_SMD:R_0402_1005Metric, symbol Device:R
- removed R65: 1k, Resistor_SMD:R_0402_1005Metric, symbol Device:R
- added C42, C43: 100nF, Capacitor_SMD:C_0603_1608Metric, symbol Device:C
- added C66: 47pF, Capacitor_SMD:C_0603_1608Metric, symbol Device:C
- added R101, R102, R103, R104, R106, R107: 22, Resistor_SMD:R_0603_1608Metric, symbol Device:R
- added R13: 1k, Resistor_SMD:R_0603_1608Metric, symbol Device:R
- added R60: 10k, Resistor_SMD:R_0603_1608Metric, symbol Device:R
- C19, C26, C33: footprint Capacitor_SMD:C_0402_1005Metric -> Capacitor_SMD:C_0603_1608Metric; Distributer Link https://www.ozdisan.com/p/smt-smd-ve-mlcc-kapasitorler-184/murata-grt155r71e104ke01d-1074547 -> https://www.ozdisan.com/p/smt-smd-ve-mlcc-kapasitorler-184/samsung-cl10b104ko8wpnc-522227; Part Number GRT155R71E104KE01D -> CL10B104KO8WPNC
- R55, R56: footprint Resistor_SMD:R_0402_1005Metric -> Resistor_SMD:R_0603_1608Metric; Distributer Link https://www.ozdisan.com/p/smt-smd-ve-cip-direncler-194/roya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 -> https://www.ozdisan.com/p/smt-smd-ve-cip-direncler-194/viki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; Part Number CQ02WGF1002TCE -> CRT03J7E1002
- R68, R69, R70, R71, R72: footprint Resistor_SMD:R_0402_1005Metric -> Resistor_SMD:R_0603_1608Metric; Distributer Link https://www.ozdisan.com/p/smt-smd-ve-cip-direncler-194/pana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 -> https://www.ozdisan.com/p/smt-smd-ve-cip-direncler-194/roya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; Part Number ERJ2RKF22R0X -> CQ03SAJ0220T5E
Connections:
- net +3.3V: now also C42.1, C43.1, C66.1, R13.1, R60.1
- net Acc_Gyro_CLK: now also R102.1, R104.2
- net Acc_Gyro_MISO: now also R101.2
- net BARO_SCK: now also R103.2
- net BARO_SS: now also R60.2
- net GND: now also C42.2, C43.2, C66.2
- net GPS_RX: now also R106.2; no longer U9.2 (TX)
- net GPS_TX: now also R107.2; no longer U9.3 (RX)
- net at U5.8 (SCLK): now also R103.1
- net at U7.14 (SCL/SCLK): now also R104.1
- net at D8.2 (A): now also R13.2
- net at U6.1 (AP_SDO/AP_AD0): now also R101.1
- net at U6.13 (AP_SCL/AP_SCLK): now also R102.2
- new net: R106.1, U9.2 (TX)
- new net: R107.1, U9.3 (RX)
- no-connect marks 9 -> 10
Other:
- note removed: "- Consider A TVS diode for RF_IN line - Select a SMA or whatever RF connector: Impedance = 50ohm"
- moved on the sheet: AE1, C16, C20, C48, D8, Q7, R68, U5, U6, U7, U9

Commit message: :)
Parts:
- U7: value ADXL375BCCZ-RL7 -> ADXL375; footprint ADXL375BCCZ_RL7:LGA_CC-14-1_ADI -> ADXL375BCCZ_RL7:LGA_CC-14-1_ADI-L; Part Number (none) -> ADXL375
Changed lines of the file:
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@@
 		(fields_autoplaced yes)
 		(property "Reference" "U7"
-			(at 110.49 113.538 0)
+			(at 95.1073 114.3 0)
 			(show_name no)
 			(do_not_autoplace no)
@@
 					(size 1.524 1.524)
 				)
+				(justify left)
 			)
 		)
-		(property "Value" "ADXL375BCCZ-RL7"
-			(at 110.49 116.078 0)
+		(property "Value" "ADXL375"
+			(at 95.1073 116.84 0)
 			(show_name no)
 			(do_not_autoplace no)
@@
 					(size 1.524 1.524)
 				)
+				(justify left)
 			)
 		)
-		(property "Footprint" "ADXL375BCCZ_RL7:LGA_CC-14-1_ADI"
+		(property "Footprint" "ADXL375BCCZ_RL7:LGA_CC-14-1_ADI-L"
 			(at 72.644 126.238 0)
 			(hide yes)
@@
 			)
 		)
-		(property "Part Number" ""
+		(property "Part Number" "ADXL375"
 			(at 94.234 133.858 0)
 			(hide yes)

Commit message: Final touches
Parts:
- U6: footprint LGA14_2P5X3X0P91_TDK -> (none)
Changed lines of the file:
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@@
 			)
 		)
-		(property "Footprint" "LGA14_2P5X3X0P91_TDK"
+		(property "Footprint" ""
 			(at 65.786 54.356 0)
 			(hide yes)

Commit message: Added MOSFET simulation files with official spice model
Parts:
- U5: Distributer Link (none) -> https://eu.mouser.com/en/ProductDetail/TE-Connectivity-Meas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; Part Number (none) -> MS561101BA03-50
- U6: footprint (none) -> ICM_42688_P:LGA14_2P5X3X0P91_TDK; Distributer Link (none) -> https://eu.mouser.com/en/ProductDetail/TDK-InvenSense/ICM-4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; Part Number (none) -> ICM-42688-P
- U7: Distributer Link (none) -> https://eu.mouser.com/en/ProductDetail/Analog-Devices/ADXL3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; Part Number ADXL375 -> ADXL375BCCZ-RL7
- U9: Distributer Link (none) -> https://eu.mouser.com/en/ProductDetail/u-blox/MAX-M10N-00B?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; Part Number (none) -> MAX-M10N-00B
Changed lines of the file:
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@@
 			)
 		)
-		(property "Description" ""
+		(property "Description" "GNSS / GPS Modules M10N LCC GNSS module, upgradeable FW in flash memory, LNA, SAW filter, TCXO"
 			(at 206.502 128.016 0)
 			(hide yes)
@@
 			)
 		)
-		(property "Distributer Link" ""
+		(property "Distributer Link" "https://eu.mouser.com/en/ProductDetail/u-blox/MAX-M10N-00B?qs=bpu3f%2FCR1jwtfwdfDBNEow%3D%3D"
 			(at 206.502 128.016 0)
 			(hide yes)
@@
 			)
 		)
-		(property "Part Number" ""
+		(property "Part Number" "MAX-M10N-00B "
 			(at 206.502 128.016 0)
 			(hide yes)
@@
 			)
 		)
+		(property "Distributer Link" "https://eu.mouser.com/en/ProductDetail/TE-Connectivity-Measurement-Specialties/MS561101BA03-50?qs=%252BgKeJhng5iV%252BnCz6Qd5iDw%3D%3D"
+			(at 215.138 62.484 0)
+			(hide yes)
+			(show_name no)
+			(do_not_autoplace no)
+			(effects
+				(font
+					(size 1.27 1.27)
+				)
+			)
+		)
+		(property "Part Number" "MS561101BA03-50"
+			(at 215.138 62.484 0)
+			(hide yes)
+			(show_name no)
+			(do_not_autoplace no)
+			(effects
+				(font
+					(size 1.27 1.27)
+				)
+			)
+		)
 		(pin "4"
 		)
@@
 			)
 		)
-		(property "Description" ""
+		(property "Description" "Accelerometers 3-Axis, 200 g Digital MEMS Accelerometer"
 			(at 94.234 133.858 0)
 			(hide yes)
@@
 			)
 		)
-		(property "Distributer Link" ""
+		(property "Distributer Link" "https://eu.mouser.com/en/ProductDetail/Analog-Devices/ADXL375BCCZ-RL7?qs=S4ILP0tmc7QIv%2F7Dk2oBJA%3D%3D"
 			(at 94.234 133.858 0)
 			(hide yes)
@@
 			)
 		)
-		(property "Part Number" "ADXL375"
+		(property "Part Number" "ADXL375BCCZ-RL7"
 			(at 94.234 133.858 0)
 			(hide yes)
@@
 			)
 		)
-		(property "Footprint" ""
+		(property "Footprint" "ICM_42688_P:LGA14_2P5X3X0P91_TDK"
 			(at 65.786 54.356 0)
 			(hide yes)
@@
 			)
 		)
-		(property "Description" ""
+		(property "Description" "SENSOR MOTION ACCELERO/GYRO 6-AXIS MEMS LGA14"
 			(at 60.96 58.42 0)
 			(hide yes)
@@
 			)
 		)
-		(property "Distributer Link" ""
+		(property "Distributer Link" "https://eu.mouser.com/en/ProductDetail/TDK-InvenSense/ICM-42688-P?qs=OlC7AqGiEDk8QrNAV728zw%3D%3D"
 			(at 60.96 58.42 0)
 			(hide yes)
@@
 			)
 		)
-		(property "Part Number" ""
+		(property "Part Number" "ICM-42688-P"
 			(at 60.96 58.42 0)
 			(hide yes)
