File: Hardware/Burocket_hardware.kicad_pcb (KiCad board)
At the start: 2 copper layers, 0 parts

Commit message: Updated schematics
Other:
- copper layers 2 -> 4
Changed lines of the file:
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@@
 	(layers
 		(0 "F.Cu" signal)
+		(4 "In1.Cu" power "GND")
+		(6 "In2.Cu" power "PWR")
 		(2 "B.Cu" signal)
 		(9 "F.Adhes" user "F.Adhesive")
@@
 		(43 "User.3" user)
 		(45 "User.4" user)
+		(47 "User.5" user)
+		(49 "User.6" user)
 	)
 	(setup
+		(stackup
+			(layer "F.SilkS"
+				(type "Top Silk Screen")
+			)
+			(layer "F.Paste"
+				(type "Top Solder Paste")
+			)
+			(layer "F.Mask"
+				(type "Top Solder Mask")
+				(thickness 0.01)
+			)
+			(layer "F.Cu"
+				(type "copper")
+				(thickness 0.035)
+			)
+			(layer "dielectric 1"
+				(type "prepreg")
+				(thickness 0.1)
+				(material "FR4")
+				(epsilon_r 4.5)
+				(loss_tangent 0.02)
+			)
+			(layer "In1.Cu"
+				(type "copper")
+				(thickness 0.035)
+			)
+			(layer "dielectric 2"
+				(type "core")
+				(thickness 1.24)
+				(material "FR4")
+				(epsilon_r 4.5)
+				(loss_tangent 0.02)
+			)
+			(layer "In2.Cu"
+				(type "copper")
+				(thickness 0.035)
+			)
+			(layer "dielectric 3"
+				(type "prepreg")
+				(thickness 0.1)
+				(material "FR4")
+				(epsilon_r 4.5)
+				(loss_tangent 0.02)
+			)
+			(layer "B.Cu"
+				(type "copper")
+				(thickness 0.035)
+			)
+			(layer "B.Mask"
+				(type "Bottom Solder Mask")
+				(thickness 0.01)
+			)
+			(layer "B.Paste"
+				(type "Bottom Solder Paste")
+			)
+			(layer "B.SilkS"
+				(type "Bottom Silk Screen")
+			)
+			(copper_finish "None")
+			(dielectric_constraints no)
+		)
 		(pad_to_mask_clearance 0)
 		(allow_soldermask_bridges_in_footprints no)

Commit message: Added New file for additional resources used, Changed LDO for lower noise, changed buck converter for higher switching speed, smaller inductance value, better transient current response
Parts:
- added AE1: Antenna, Connector_Coaxial:SMA_Amphenol_132134-10_Vertical, F.Cu at (152.9, 95.0)
- added BT1: Battery, Connector_AMASS:AMASS_XT60-F_1x02_P7.20mm_Vertical, F.Cu at (141.9, 53.4)
- added BZ1: Buzzer, footprints:Buzzer_typeshit, F.Cu at (130.7, 75.3)
- added C1: 100nF, Capacitor_SMD:C_0402_1005Metric, F.Cu at (127.6, 63.7)
- added C10: 20pF, Capacitor_SMD:C_0603_1608Metric, F.Cu at (110.8, 64.0)
- added C11: 100nF, Capacitor_SMD:C_0402_1005Metric, F.Cu at (133.3, 65.7)
- added C12: 2.2uF, Capacitor_SMD:C_0603_1608Metric, F.Cu at (110.8, 66.5)
- added C13: 2.2uF, Capacitor_SMD:C_0603_1608Metric, F.Cu at (110.8, 69.0)
- added C14: 2.2uF, Capacitor_SMD:C_0603_1608Metric, F.Cu at (110.8, 71.5)
- added C15: 100nF, Capacitor_SMD:C_0402_1005Metric, F.Cu at (110.2, 83.3)
- added C16: 2.2uF, Capacitor_SMD:C_0603_1608Metric, F.Cu at (159.5, 91.7)
- added C17: 100nF, Capacitor_SMD:C_0402_1005Metric, F.Cu at (55.4, 65.1)
- added C18: 20pF, Capacitor_SMD:C_0603_1608Metric, F.Cu at (110.8, 74.1)
- added C19: 100nF, Capacitor_SMD:C_0402_1005Metric, F.Cu at (138.2, 95.3)
- added C2: 100nF, Capacitor_SMD:C_0402_1005Metric, F.Cu at (127.6, 65.7)
- added C20: 2.2uF, Capacitor_SMD:C_0603_1608Metric, F.Cu at (159.5, 94.2)
- added C21: 2.2uF, Capacitor_SMD:C_0603_1608Metric, F.Cu at (168.4, 92.6)
- added C22: 100nF, Capacitor_SMD:C_0402_1005Metric, F.Cu at (184.1, 81.2)
- added C23: 100nF, Capacitor_SMD:C_0402_1005Metric, F.Cu at (151.4, 67.7)
- added C24: 0.1nF, Capacitor_SMD:C_0402_1005Metric, F.Cu at (151.4, 69.7)
- added C25: 47uF, Capacitor_SMD:C_1210_3225Metric, F.Cu at (157.1, 54.9)
- added C26: 100nF, Capacitor_SMD:C_0402_1005Metric, F.Cu at (138.2, 97.3)
- added C27: 2.2uF, Capacitor_SMD:C_0402_1005Metric, F.Cu at (110.2, 85.3)
- added C28: 100nF, Capacitor_SMD:C_0402_1005Metric, F.Cu at (110.2, 87.3)
- added C29: 100nF, Capacitor_SMD:C_0402_1005Metric, F.Cu at (110.2, 89.2)
- added C3: 100nF, Capacitor_SMD:C_0402_1005Metric, F.Cu at (127.6, 67.7)
- added C30: 100nF, Capacitor_SMD:C_0402_1005Metric, F.Cu at (221.1, 71.0)
- added C31: 100nF, Capacitor_SMD:C_0402_1005Metric, F.Cu at (226.3, 65.3)
- added C32: 0.1nF, Capacitor_SMD:C_0402_1005Metric, F.Cu at (138.2, 99.3)
- added C33: 100nF, Capacitor_SMD:C_0402_1005Metric, F.Cu at (138.2, 101.3)
- added C34: 100uF, Capacitor_Tantalum_SMD:CP_EIA-6032-20_AVX-F, F.Cu at (167.9, 99.1)
- added C35: 2.2uF, Capacitor_SMD:C_0603_1608Metric, F.Cu at (162.7, 71.6)
- added C36: 100nF, Capacitor_SMD:C_0402_1005Metric, F.Cu at (110.2, 91.2)
- added C37: 100nF, Capacitor_SMD:C_0402_1005Metric, F.Cu at (110.2, 93.2)
- added C38: 22uF, Capacitor_SMD:C_0805_2012Metric, F.Cu at (139.0, 60.1)
- added C39: 100nF, Capacitor_SMD:C_0402_1005Metric, F.Cu at (110.2, 95.1)
- added C4: 100nF, Capacitor_SMD:C_0402_1005Metric, F.Cu at (130.4, 63.7)
- added C40: 100nF, Capacitor_SMD:C_0402_1005Metric, F.Cu at (151.4, 75.6)
- added C41: 22uF, Capacitor_SMD:C_0805_2012Metric, F.Cu at (139.0, 63.1)
- added C42: 22uF, Capacitor_SMD:C_0805_2012Metric, F.Cu at (139.0, 66.1)
- added C43: 22uF, Capacitor_SMD:C_0805_2012Metric, F.Cu at (139.0, 69.1)
- added C44: 22uF, Capacitor_SMD:C_0805_2012Metric, F.Cu at (139.0, 72.1)
- added C45: 22uF, Capacitor_SMD:C_0805_2012Metric, F.Cu at (132.2, 70.2)
- added C46: 22uF, Capacitor_SMD:C_0805_2012Metric, F.Cu at (128.3, 83.8)
- added C47: 22uF, Capacitor_SMD:C_0805_2012Metric, F.Cu at (128.3, 86.8)
- added C48: 22uF, Capacitor_SMD:C_0805_2012Metric, F.Cu at (150.6, 101.1)
- added C49: 100uF, Capacitor_Tantalum_SMD:CP_EIA-6032-20_AVX-F, F.Cu at (167.9, 103.9)
- added C5: 100nF, Capacitor_SMD:C_0402_1005Metric, F.Cu at (130.4, 65.7)
- added C50: 100uF, Capacitor_Tantalum_SMD:CP_EIA-6032-20_AVX-F, F.Cu at (167.9, 108.6)
- added C51: 100nF, Capacitor_SMD:C_0402_1005Metric, F.Cu at (173.6, 97.7)
- added C52: 2.2uF, Capacitor_SMD:C_0603_1608Metric, F.Cu at (162.7, 74.1)
- added C6: 100nF, Capacitor_SMD:C_0402_1005Metric, F.Cu at (130.4, 67.7)
- added C7: 100nF, Capacitor_SMD:C_0402_1005Metric, F.Cu at (133.3, 63.7)
- added C8: 100nF, Capacitor_SMD:C_0402_1005Metric, F.Cu at (138.2, 91.4)
- added C9: 100nF, Capacitor_SMD:C_0402_1005Metric, F.Cu at (138.2, 93.4)
- added D1: Blue_LED, Capacitor_SMD:C_0603_1608Metric, F.Cu at (110.8, 76.6)
- added D2: Red LED, Capacitor_SMD:C_0603_1608Metric, F.Cu at (110.8, 79.1)
- added D3: ESD321DYAR, Diode_SMD:D_SOD-523, F.Cu at (172.3, 90.0)
- added D4: Green LED, LED_SMD:LED_0603_1608Metric, F.Cu at (168.5, 90.1)
- added D5: 1N4448W, Diode_SMD:Nexperia_CFP3_SOD-123W, F.Cu at (120.2, 77.1)
- added D6: 1N4148W, Diode_SMD:D_SOD-123, F.Cu at (120.3, 70.4)
- added D7: 1N4148W, Diode_SMD:D_SOD-123, F.Cu at (120.3, 73.8)
- added D8: Red LED, Capacitor_SMD:C_0603_1608Metric, F.Cu at (159.5, 96.7)
- added J1: USB4105-GF-A-120, USB4105-GF-A-120:GCT_USB4105-GF-A-120, F.Cu at (192.8, 77.5)
- added J3: 1040310811, Molex 1040310811:104031-0811_MOL, F.Cu at (68.8, 75.3)
- added J5: Conn_01x05_Pin, Connector_PinHeader_2.54mm:PinHeader_1x05_P2.54mm_Vertical, F.Cu at (81.9, 74.7)
- added J8: Conn_01x07_Pin, footprints:E32-900T30D, F.Cu at (92.8, 69.5)
- added L1: 9.1uH, Inductor_SMD_Wurth:L_Wurth_WE-PDF-1045, F.Cu at (159.4, 64.4)
- added Q1: BC847, Package_TO_SOT_SMD:SOT-323_SC-70, F.Cu at (125.2, 59.8)
- added Q7: BCR116, Package_TO_SOT_SMD:SOT-23-3, F.Cu at (157.0, 87.6)
- added R10: 1k, Resistor_SMD:R_0402_1005Metric, F.Cu at (121.8, 63.8)
- added R11: 1k, Resistor_SMD:R_0402_1005Metric, F.Cu at (121.8, 65.7)
- added R14: 22, Resistor_SMD:R_0402_1005Metric, F.Cu at (113.1, 97.1)
- added R16: 10k, Resistor_SMD:R_0402_1005Metric, F.Cu at (113.1, 99.1)
- added R17: 10k, Resistor_SMD:R_0402_1005Metric, F.Cu at (113.1, 101.1)
- added R18: 10k, Resistor_SMD:R_0402_1005Metric, F.Cu at (113.1, 103.1)
- added R19: 10k, Resistor_SMD:R_0402_1005Metric, F.Cu at (116.0, 97.1)
- added R2: 5.1k, Resistor_SMD:R_0402_1005Metric, F.Cu at (165.0, 89.8)
- added R20: 10k, Resistor_SMD:R_0402_1005Metric, F.Cu at (116.0, 99.1)
- added R21: 100k, Resistor_SMD:R_0402_1005Metric, F.Cu at (142.7, 67.7)
- added R22: 13.7K, Resistor_SMD:R_0402_1005Metric, F.Cu at (142.7, 69.7)
- added R23: 412k, Resistor_SMD:R_0402_1005Metric, F.Cu at (142.7, 71.7)
- added R24: 97.6K, Resistor_SMD:R_0402_1005Metric, F.Cu at (142.7, 73.7)
- added R25: 1k, Resistor_SMD:R_0402_1005Metric, F.Cu at (165.0, 93.7)
- added R26: 10k, Resistor_SMD:R_0402_1005Metric, F.Cu at (121.8, 67.7)
- added R27: 4.7, Resistor_SMD:R_0402_1005Metric, F.Cu at (124.7, 63.8)
- added R28: 10k, Resistor_SMD:R_0402_1005Metric, F.Cu at (59.4, 65.3)
- added R29: 48.7K, Resistor_SMD:R_0402_1005Metric, F.Cu at (142.7, 75.7)
- added R3: 5.1k, Resistor_SMD:R_0402_1005Metric, F.Cu at (165.0, 91.8)
- added R30: 48.7K, Resistor_SMD:R_0402_1005Metric, F.Cu at (145.6, 67.7)
- added R31: 48.7K, Resistor_SMD:R_0402_1005Metric, F.Cu at (145.6, 69.7)
- added R32: 28k, Resistor_SMD:R_0402_1005Metric, F.Cu at (145.6, 71.7)
- added R35: 4.7, Resistor_SMD:R_0402_1005Metric, F.Cu at (116.0, 101.1)
- added R36: 10k, Resistor_SMD:R_0402_1005Metric, F.Cu at (145.6, 73.7)
- added R37: 10k, Resistor_SMD:R_0402_1005Metric, F.Cu at (145.6, 75.7)
- added R38: 10k, Resistor_SMD:R_0402_1005Metric, F.Cu at (148.5, 67.7)
- added R4: 5.1k, Resistor_SMD:R_0402_1005Metric, F.Cu at (118.9, 63.8)
- added R41: 4.7, Resistor_SMD:R_0402_1005Metric, F.Cu at (116.0, 103.1)
- added R44: 4.7, Resistor_SMD:R_0402_1005Metric, F.Cu at (119.0, 97.1)
- added R5: 5.1k, Resistor_SMD:R_0402_1005Metric, F.Cu at (118.9, 65.7)
- added R52: 4.7, Resistor_SMD:R_0402_1005Metric, F.Cu at (119.0, 99.1)
- added R53: 10k, Resistor_SMD:R_0402_1005Metric, F.Cu at (124.7, 67.7)
- added R54: 10k, Resistor_SMD:R_0402_1005Metric, F.Cu at (141.1, 91.4)
- added R55: 10k, Resistor_SMD:R_0402_1005Metric, F.Cu at (141.1, 93.4)
- added R56: 10k, Resistor_SMD:R_0402_1005Metric, F.Cu at (141.1, 95.4)
- added R57: 22, Resistor_SMD:R_0402_1005Metric, F.Cu at (141.1, 97.4)
- added R58: 22, Resistor_SMD:R_0402_1005Metric, F.Cu at (141.1, 99.4)
- added R59: 22, Resistor_SMD:R_0402_1005Metric, F.Cu at (144.0, 91.4)
- added R60: 4.7, Resistor_SMD:R_0402_1005Metric, F.Cu at (208.7, 67.0)
- added R61: 4.7, Resistor_SMD:R_0402_1005Metric, F.Cu at (208.7, 69.0)
- added R62: 10k, Resistor_SMD:R_0402_1005Metric, F.Cu at (119.0, 101.1)
- added R63: 22Ω, Resistor_SMD:R_0402_1005Metric, F.Cu at (119.0, 103.1)
- added R64: 10k, Resistor_SMD:R_0402_1005Metric, F.Cu at (121.9, 97.1)
- added R65: 1k, Resistor_SMD:R_0402_1005Metric, F.Cu at (144.0, 93.4)
- added R66: 28k, Resistor_SMD:R_0402_1005Metric, F.Cu at (121.9, 99.1)
- added R67: 22, Resistor_SMD:R_0402_1005Metric, F.Cu at (144.0, 95.4)
- added R68: 22, Resistor_SMD:R_0402_1005Metric, F.Cu at (144.0, 97.4)
- added R69: 22, Resistor_SMD:R_0402_1005Metric, F.Cu at (144.0, 99.4)
- added R70: 22, Resistor_SMD:R_0402_1005Metric, F.Cu at (146.9, 91.4)
- added R71: 22, Resistor_SMD:R_0402_1005Metric, F.Cu at (146.9, 93.4)
- added R72: 22, Resistor_SMD:R_0402_1005Metric, F.Cu at (146.9, 95.4)
- added R73: 22Ω, Resistor_SMD:R_0402_1005Metric, F.Cu at (121.9, 101.1)
- added R74: 22Ω, Resistor_SMD:R_0402_1005Metric, F.Cu at (121.9, 103.1)
- added R9: 1k, Resistor_SMD:R_0402_1005Metric, F.Cu at (118.9, 67.7)
- added R_Shunt1: 5m, Resistor_SMD:R_1206_3216Metric, F.Cu at (162.8, 54.4)
- added SW1: SW_Push, Button_Switch_SMD:SW_SPST_PTS810, F.Cu at (126.6, 71.1)
- added SW2: SW_SPDT, Button_Switch_SMD:SW_SPDT_CK_JS102011SAQN, F.Cu at (57.0, 59.8)
- added U1: STM32F405RGT6, Package_QFP:LQFP-64_10x10mm_P0.5mm, F.Cu at (60.5, 92.0)
- added U10: INA226, Package_SO:TSSOP-10_3x3mm_P0.5mm, F.Cu at (217.3, 69.8)
- added U11: W25Q128JVS, Package_SO:SOIC-8_5.3x5.3mm_P1.27mm, F.Cu at (66.9, 107.4)
- added U2: TPS54302, TPS54302DDCR:SOT95P280X110-6N, F.Cu at (157.4, 50.5)
- added U3: LD1086DT33TR, Package_TO_SOT_SMD:TO-252-2, F.Cu at (148.1, 62.7)
- added U4: TPD2EUSB30DRTR, Package_TO_SOT_SMD:Texas_DRT-3, F.Cu at (172.1, 92.4)
- added U5: MS5611-01BA, Package_LGA:LGA-8_3x5mm_P1.25mm, F.Cu at (152.1, 82.2)
- added U6: ICM-42688-P, ICM_42688_P:LGA14_2P5X3X0P91_TDK, F.Cu at (151.9, 87.6)
- added U7: ADXL375BCCZ-RL7, ADXL375BCCZ_RL7:LGA_CC-14-1_ADI, F.Cu at (157.2, 82.0)
- added U8: TPS2121RUXR, footprints.ugly:RUX0012A, F.Cu at (161.8, 50.3)
- added U9: MAX-M10N, RF_GPS:ublox_MAX, F.Cu at (143.2, 84.6)
- added Y2: 25MHz, Crystal:Crystal_SMD_3225-4Pin_3.2x2.5mm, F.Cu at (125.8, 75.8)

Commit message: Added Impedance matching calculations, finished buck converter calculations, finalized buzzer circuitry
Parts:
- removed AE1: Antenna, Connector_Coaxial:SMA_Amphenol_132134-10_Vertical
- removed BT1: Battery, Connector_AMASS:AMASS_XT60-F_1x02_P7.20mm_Vertical
- removed BZ1: Buzzer, footprints:Buzzer_typeshit
- removed C1, C11, C15, C17, C19, C2, C22, C23, C26, C28, C29, C3, C30, C31, C33, C36, C37, C39, C4, C40, C5, C51, C6, C7, C8, C9: 100nF, Capacitor_SMD:C_0402_1005Metric
- removed C10, C18: 20pF, Capacitor_SMD:C_0603_1608Metric
- removed C12, C13, C14, C16, C20, C21, C35, C52: 2.2uF, Capacitor_SMD:C_0603_1608Metric
- removed C24, C32: 0.1nF, Capacitor_SMD:C_0402_1005Metric
- removed C25: 47uF, Capacitor_SMD:C_1210_3225Metric
- removed C27: 2.2uF, Capacitor_SMD:C_0402_1005Metric
- removed C34, C49, C50: 100uF, Capacitor_Tantalum_SMD:CP_EIA-6032-20_AVX-F
- removed C38, C41, C42, C43, C44, C45, C46, C47, C48: 22uF, Capacitor_SMD:C_0805_2012Metric
- removed D1: Blue_LED, Capacitor_SMD:C_0603_1608Metric
- removed D2, D8: Red LED, Capacitor_SMD:C_0603_1608Metric
- removed D3: ESD321DYAR, Diode_SMD:D_SOD-523
- removed D4: Green LED, LED_SMD:LED_0603_1608Metric
- removed D5: 1N4448W, Diode_SMD:Nexperia_CFP3_SOD-123W
- removed D6, D7: 1N4148W, Diode_SMD:D_SOD-123
- removed J1: USB4105-GF-A-120, USB4105-GF-A-120:GCT_USB4105-GF-A-120
- removed J3: 1040310811, Molex 1040310811:104031-0811_MOL
- removed J5: Conn_01x05_Pin, Connector_PinHeader_2.54mm:PinHeader_1x05_P2.54mm_Vertical
- removed J8: Conn_01x07_Pin, footprints:E32-900T30D
- removed L1: 9.1uH, Inductor_SMD_Wurth:L_Wurth_WE-PDF-1045
- removed Q1: BC847, Package_TO_SOT_SMD:SOT-323_SC-70
- removed Q7: BCR116, Package_TO_SOT_SMD:SOT-23-3
- removed R10, R11, R25, R65, R9: 1k, Resistor_SMD:R_0402_1005Metric
- removed R14, R57, R58, R59, R67, R68, R69, R70, R71, R72: 22, Resistor_SMD:R_0402_1005Metric
- removed R16, R17, R18, R19, R20, R26, R28, R36, R37, R38, R53, R54, R55, R56, R62, R64: 10k, Resistor_SMD:R_0402_1005Metric
- removed R2, R3, R4, R5: 5.1k, Resistor_SMD:R_0402_1005Metric
- removed R21: 100k, Resistor_SMD:R_0402_1005Metric
- removed R22: 13.7K, Resistor_SMD:R_0402_1005Metric
- removed R23: 412k, Resistor_SMD:R_0402_1005Metric
- removed R24: 97.6K, Resistor_SMD:R_0402_1005Metric
- removed R27, R35, R41, R44, R52, R60, R61: 4.7, Resistor_SMD:R_0402_1005Metric
- removed R29, R30, R31: 48.7K, Resistor_SMD:R_0402_1005Metric
- removed R32, R66: 28k, Resistor_SMD:R_0402_1005Metric
- removed R63, R73, R74: 22Ω, Resistor_SMD:R_0402_1005Metric
- removed R_Shunt1: 5m, Resistor_SMD:R_1206_3216Metric
- removed SW1: SW_Push, Button_Switch_SMD:SW_SPST_PTS810
- removed SW2: SW_SPDT, Button_Switch_SMD:SW_SPDT_CK_JS102011SAQN
- removed U1: STM32F405RGT6, Package_QFP:LQFP-64_10x10mm_P0.5mm
- removed U10: INA226, Package_SO:TSSOP-10_3x3mm_P0.5mm
- removed U11: W25Q128JVS, Package_SO:SOIC-8_5.3x5.3mm_P1.27mm
- removed U2: TPS54302, TPS54302DDCR:SOT95P280X110-6N
- removed U3: LD1086DT33TR, Package_TO_SOT_SMD:TO-252-2
- removed U4: TPD2EUSB30DRTR, Package_TO_SOT_SMD:Texas_DRT-3
- removed U5: MS5611-01BA, Package_LGA:LGA-8_3x5mm_P1.25mm
- removed U6: ICM-42688-P, ICM_42688_P:LGA14_2P5X3X0P91_TDK
- removed U7: ADXL375BCCZ-RL7, ADXL375BCCZ_RL7:LGA_CC-14-1_ADI
- removed U8: TPS2121RUXR, footprints.ugly:RUX0012A
- removed U9: MAX-M10N, RF_GPS:ublox_MAX
- removed Y2: 25MHz, Crystal:Crystal_SMD_3225-4Pin_3.2x2.5mm

Commit message: Purged heavy binaries and updated gitignore
Parts:
- added BT1: Battery, Connector_AMASS:AMASS_XT60-M_1x02_P7.20mm_Vertical, F.Cu at (109.9, 111.2)
- added BZ1: Buzzer, footprints:Buzzer_typeshit, F.Cu at (94.6, 72.0)
- added C11: 100nF, Capacitor_SMD:C_0603_1608Metric, B.Cu at (80.4, 94.0)
- added C12: 2.2uF, Capacitor_SMD:C_0603_1608Metric, B.Cu at (95.9, 95.4)
- added C13: 2.2uF, Capacitor_SMD:C_0603_1608Metric, B.Cu at (100.6, 83.2)
- added C14: 2.2uF, Capacitor_SMD:C_0603_1608Metric, F.Cu at (81.8, 88.1)
- added C15: 100nF, Capacitor_SMD:C_0603_1608Metric, F.Cu at (100.9, 97.8)
- added C16: 2.2uF, Capacitor_SMD:C_0603_1608Metric, F.Cu at (91.8, 100.5)
- added C17: 100nF, Capacitor_SMD:C_0603_1608Metric, F.Cu at (95.1, 67.5)
- added C18: 10pF, Capacitor_SMD:C_0603_1608Metric, B.Cu at (83.4, 84.2)
- added C19: 100nF, Capacitor_SMD:C_0603_1608Metric, F.Cu at (83.2, 102.5)
- added C20: 2.2uF, Capacitor_SMD:C_0603_1608Metric, F.Cu at (83.2, 104.0)
- added C21: 100nF, Capacitor_SMD:C_0603_1608Metric, B.Cu at (89.7, 79.5)
- added C22: 100nF, Capacitor_SMD:C_0603_1608Metric, F.Cu at (115.7, 86.5)
- added C23: 100nF, Capacitor_SMD:C_0603_1608Metric, B.Cu at (97.0, 83.7)
- added C24: 2.2uF, Capacitor_SMD:C_0603_1608Metric, F.Cu at (83.6, 81.4)
- added C25: 100nF, Capacitor_SMD:C_0603_1608Metric, B.Cu at (94.5, 91.4)
- added C26: 100nF, Capacitor_SMD:C_0603_1608Metric, F.Cu at (93.3, 103.6)
- added C27: 2.2uF, Capacitor_SMD:C_0603_1608Metric, B.Cu at (108.5, 68.7)
- added C28: 100nF, Capacitor_SMD:C_0603_1608Metric, B.Cu at (96.0, 80.8)
- added C29: 100nF, Capacitor_SMD:C_0603_1608Metric, B.Cu at (88.6, 84.6)
- added C30: 100nF, Capacitor_SMD:C_0603_1608Metric, B.Cu at (133.9, 116.0)
- added C31: 100nF, Capacitor_SMD:C_0603_1608Metric, B.Cu at (129.1, 109.1)
- added C32: 100nF, Capacitor_SMD:C_0603_1608Metric, B.Cu at (126.8, 115.6)
- added C33: 100nF, Capacitor_SMD:C_0603_1608Metric, F.Cu at (83.6, 79.9)
- added C34: 100uF, Capacitor_Tantalum_SMD:CP_EIA-6032-20_AVX-F, F.Cu at (56.7, 71.8)
- added C35: 2.2uF, Capacitor_SMD:C_0603_1608Metric, B.Cu at (120.4, 90.2)
- added C36: 100nF, Capacitor_SMD:C_0603_1608Metric, B.Cu at (91.6, 85.1)
- added C37: 100nF, Capacitor_SMD:C_0603_1608Metric, B.Cu at (89.1, 87.6)
- added C38: 100nF, Capacitor_SMD:C_0603_1608Metric, B.Cu at (88.6, 92.4)
- added C39: 100nF, Capacitor_SMD:C_0603_1608Metric, B.Cu at (85.1, 89.9)
- added C40: 100nF, Capacitor_SMD:C_0603_1608Metric, B.Cu at (85.4, 80.7)
- added C41: 100nF, Capacitor_SMD:C_0603_1608Metric, F.Cu at (84.1, 88.8)
- added C42: 100nF, Capacitor_SMD:C_0603_1608Metric, B.Cu at (84.0, 100.0)
- added C43: 100nF, Capacitor_SMD:C_0603_1608Metric, F.Cu at (86.9, 105.5)
- added C44: 100nF, Capacitor_SMD:C_0603_1608Metric, F.Cu at (114.2, 101.8)
- added C45: 22uF, Capacitor_SMD:C_0805_2012Metric, B.Cu at (87.2, 80.5)
- added C46: 22uF, Capacitor_SMD:C_0805_2012Metric, F.Cu at (89.2, 71.7)
- added C47: 2.2uF, Capacitor_SMD:C_0603_1608Metric, F.Cu at (99.4, 97.8)
- added C48: 22uF, Capacitor_SMD:C_0805_2012Metric, B.Cu at (83.5, 74.5)
- added C49: 100uF, Capacitor_Tantalum_SMD:CP_EIA-6032-20_AVX-F, F.Cu at (56.7, 68.0)
- added C50: 100uF, Capacitor_Tantalum_SMD:CP_EIA-6032-20_AVX-F, F.Cu at (56.7, 64.0)
- added C51: 100nF, Capacitor_SMD:C_0603_1608Metric, B.Cu at (57.6, 77.6)
- added C52: 22uF, Capacitor_SMD:C_0805_2012Metric, F.Cu at (115.5, 88.3)
- added C53: 22uF, Capacitor_SMD:C_0805_2012Metric, F.Cu at (107.9, 75.9)
- added C54: 2.2uF, Capacitor_SMD:C_0603_1608Metric, B.Cu at (107.3, 83.4)
- added C55: 2.2uF, Capacitor_SMD:C_0603_1608Metric, F.Cu at (110.5, 76.7)
- added C56: 100nF, Capacitor_SMD:C_0603_1608Metric, F.Cu at (112.1, 76.7)
- added C57: 22uF, Capacitor_SMD:C_0805_2012Metric, F.Cu at (111.2, 81.8)
- added C58: 100nF, Capacitor_SMD:C_0603_1608Metric, B.Cu at (107.8, 81.9)
- added C59: 100nF, Capacitor_SMD:C_0603_1608Metric, F.Cu at (112.2, 96.8)
- added C60: 100nF, Capacitor_SMD:C_0603_1608Metric, F.Cu at (113.0, 94.5)
- added C61: 10pF, Capacitor_SMD:C_0603_1608Metric, B.Cu at (82.0, 85.6)
- added C62: 22uF, Capacitor_SMD:C_0805_2012Metric, B.Cu at (108.4, 70.5)
- added C63: 100nF, Capacitor_SMD:C_0603_1608Metric, F.Cu at (93.3, 100.5)
- added C64: 47uF, Capacitor_SMD:C_1210_3225Metric, F.Cu at (122.4, 103.2)
- added C65: 47pF, Capacitor_SMD:C_0603_1608Metric, F.Cu at (109.9, 95.1)
- added C66: 47pF, Capacitor_SMD:C_0603_1608Metric, B.Cu at (83.8, 77.8)
- added C67: 100nF, Capacitor_SMD:C_0603_1608Metric, B.Cu at (83.8, 76.2)
- added C68: 100nF, Capacitor_SMD:C_0603_1608Metric, F.Cu at (121.7, 62.7)
- added C69: 47uF, Capacitor_SMD:C_1210_3225Metric, F.Cu at (119.1, 103.2)
- added C70: 47uF, Capacitor_SMD:C_1210_3225Metric, F.Cu at (115.0, 104.1)
- added D1: Blue_LED, Capacitor_SMD:C_0603_1608Metric, F.Cu at (78.3, 84.2)
- added D2: Red LED, Capacitor_SMD:C_0603_1608Metric, F.Cu at (78.3, 85.7)
- added D3: ESD321DYAR, Diode_SMD:D_SOD-523, F.Cu at (115.9, 85.0)
- added D4: Green LED, LED_SMD:LED_0603_1608Metric, F.Cu at (119.3, 75.5)
- added D5: 1N4448W, Diode_SMD:Nexperia_CFP3_SOD-123W, F.Cu at (97.1, 71.7)
- added D6: 1N4148, Diode_SMD:D_SOD-523, F.Cu at (91.5, 72.7)
- added D7: 1N4148, Diode_SMD:D_SOD-523, F.Cu at (91.5, 71.2)
- added D8: Red LED, Capacitor_SMD:C_0603_1608Metric, F.Cu at (71.1, 68.7)
- added FB1: FerriteBead, Resistor_SMD:R_0603_1608Metric, F.Cu at (81.8, 89.6)
- added H1: MountingHole_Pad, MountingHole:MountingHole_2.2mm_M2_Pad_Via, F.Cu at (149.4, 61.8)
- added H2: MountingHole_Pad, MountingHole:MountingHole_2.2mm_M2_Pad_Via, F.Cu at (149.4, 67.7)
- added H3: MountingHole_Pad, MountingHole:MountingHole_2.2mm_M2_Pad_Via, F.Cu at (149.4, 73.7)
- added H4: MountingHole_Pad, MountingHole:MountingHole_2.2mm_M2_Pad_Via, F.Cu at (149.4, 79.6)
- added J1: USB4105-GF-A-120, USB4105-GF-A-120:GCT_USB4105-GF-A-120, F.Cu at (123.4, 83.1)
- added J10: Conn_01x02, ICM_42688_P:E-match_Solder, F.Cu at (88.5, 115.1)
- added J11: Conn_01x02, ICM_42688_P:E-match_Solder, F.Cu at (102.7, 114.8)
- added J2: Conn_Coaxial, Connector_Coaxial:SMA_Amphenol_132134-10_Vertical, F.Cu at (84.8, 62.9)
- added J4: 1040310811, Molex 1040310811:104031-0811_MOL, F.Cu at (109.8, 64.0)
- added J5: Conn_01x05_Pin, Connector_PinHeader_2.54mm:PinHeader_1x05_P2.54mm_Vertical, F.Cu at (124.3, 61.2)
- added J7: Conn_01x02, ICM_42688_P:E-match_Solder, F.Cu at (95.7, 115.0)
- added J8: Conn_01x07_Pin, footprints:E32-900T30D, F.Cu at (65.9, 86.1)
- added J9: Conn_01x02, ICM_42688_P:E-match_Solder, F.Cu at (81.4, 115.3)
- added L3: 6.8uH, Inductor_SMD:L_Wuerth_XHMI-6060, F.Cu at (118.1, 97.4)
- added Q1: BC847, Package_TO_SOT_SMD:SOT-323_SC-70, F.Cu at (99.8, 73.8)
- added Q11: IRLML0030, Package_TO_SOT_SMD:SOT-23, F.Cu at (87.3, 111.7)
- added Q6: IRLML0030, Package_TO_SOT_SMD:SOT-23, F.Cu at (94.5, 111.5)
- added Q7: BCR116, Package_TO_SOT_SMD:SOT-23-3, F.Cu at (74.7, 67.2)
- added Q8: IRLML0030, Package_TO_SOT_SMD:SOT-23, F.Cu at (80.5, 111.8)
- added Q9: IRLML0030, Package_TO_SOT_SMD:SOT-23, F.Cu at (101.5, 111.3)
- added R10: 1k, Resistor_SMD:R_0603_1608Metric, B.Cu at (78.3, 84.2)
- added R100: 10k, Resistor_SMD:R_0603_1608Metric, B.Cu at (128.3, 121.2)
- added R101: 22, Resistor_SMD:R_0603_1608Metric, F.Cu at (79.5, 99.3)
- added R102: 22, Resistor_SMD:R_0603_1608Metric, F.Cu at (94.4, 95.4)
- added R105: 22, Resistor_SMD:R_0603_1608Metric, F.Cu at (96.0, 76.6)
- added R106: 22, Resistor_SMD:R_0603_1608Metric, F.Cu at (78.6, 80.7)
- added R107: 22, Resistor_SMD:R_0603_1608Metric, F.Cu at (90.5, 76.9)
- added R108: 22, Resistor_SMD:R_0603_1608Metric, F.Cu at (63.9, 72.2)
- added R109: 22, Resistor_SMD:R_0603_1608Metric, F.Cu at (110.4, 72.6)
- added R11: 1k, Resistor_SMD:R_0603_1608Metric, F.Cu at (96.7, 74.6)
- added R110: 22, Resistor_SMD:R_0603_1608Metric, F.Cu at (112.0, 72.6)
- added R111: 22, Resistor_SMD:R_0603_1608Metric, F.Cu at (113.5, 72.5)
- added R112: 22, Resistor_SMD:R_0603_1608Metric, F.Cu at (104.8, 72.6)
- added R113: 22, Resistor_SMD:R_0603_1608Metric, F.Cu at (106.3, 72.6)
- added R114: 22, Resistor_SMD:R_0603_1608Metric, F.Cu at (120.9, 71.5)
- added R115: 22, Resistor_SMD:R_0603_1608Metric, F.Cu at (120.9, 68.8)
- added R116: 22, Resistor_SMD:R_0603_1608Metric, F.Cu at (120.9, 66.3)
- added R117: 22, Resistor_SMD:R_0603_1608Metric, F.Cu at (100.7, 87.1)
- added R118: 22, Resistor_SMD:R_0603_1608Metric, F.Cu at (98.1, 92.2)
- added R119: 22, Resistor_SMD:R_0603_1608Metric, F.Cu at (89.4, 95.3)
- added R12: 1k, Resistor_SMD:R_0603_1608Metric, B.Cu at (78.3, 85.7)
- added R120: 22, Resistor_SMD:R_0603_1608Metric, F.Cu at (91.4, 95.4)
- added R121: 22, Resistor_SMD:R_0603_1608Metric, F.Cu at (92.8, 95.3)
- added R122: 22, Resistor_SMD:R_0603_1608Metric, F.Cu at (66.7, 72.1)
- added R13: 1k, Resistor_SMD:R_0603_1608Metric, F.Cu at (71.0, 67.1)
- added R14: 220, Resistor_SMD:R_0603_1608Metric, F.Cu at (92.4, 76.9)
- added R15: 1k, Resistor_SMD:R_0603_1608Metric, F.Cu at (119.3, 77.0)
- added R16: 220, Resistor_SMD:R_0603_1608Metric, F.Cu at (81.3, 80.7)
- added R17: 4.7k, Resistor_SMD:R_0603_1608Metric, F.Cu at (71.6, 72.1)
- added R18: 4.7k, Resistor_SMD:R_0603_1608Metric, F.Cu at (69.1, 72.2)
- added R27: 22, Resistor_SMD:R_0603_1608Metric, F.Cu at (91.7, 69.8)
- added R28: 4.7, Resistor_SMD:R_0603_1608Metric, B.Cu at (128.4, 111.4)
- added R29: 48.7K, Resistor_SMD:R_0603_1608Metric, F.Cu at (107.9, 88.4)
- added R30: 48.7K, Resistor_SMD:R_0603_1608Metric, F.Cu at (107.9, 85.4)
- added R31: 48.7K, Resistor_SMD:R_0603_1608Metric, B.Cu at (120.4, 91.8)
- added R32: 28k, Resistor_SMD:R_0603_1608Metric, F.Cu at (107.9, 91.5)
- added R33: 4.7, Resistor_SMD:R_0603_1608Metric, B.Cu at (129.9, 111.4)
- added R34: 4.7, Resistor_SMD:R_0603_1608Metric, F.Cu at (113.7, 96.8)
- added R35: 4.7, Resistor_SMD:R_0603_1608Metric, B.Cu at (91.7, 83.6)
- added R36: 4.7, Resistor_SMD:R_0603_1608Metric, B.Cu at (85.1, 88.4)
- added R37: 4.7, Resistor_SMD:R_0603_1608Metric, B.Cu at (88.6, 83.1)
- added R38: 4.7, Resistor_SMD:R_0603_1608Metric, B.Cu at (90.6, 87.6)
- added R4: 4.7k, Resistor_SMD:R_0603_1608Metric, B.Cu at (132.5, 121.3)
- added R40: 28k, Resistor_SMD:R_0603_1608Metric, F.Cu at (118.1, 61.6)
- added R41: 28k, Resistor_SMD:R_0603_1608Metric, F.Cu at (93.1, 114.0)
- added R43: 28k, Resistor_SMD:R_0603_1608Metric, F.Cu at (100.1, 113.8)
- added R44: 28k, Resistor_SMD:R_0603_1608Metric, F.Cu at (85.9, 114.1)
- added R45: 300, Resistor_SMD:R_0603_1608Metric, F.Cu at (96.8, 109.1)
- added R46: 28k, Resistor_SMD:R_0603_1608Metric, F.Cu at (78.8, 114.2)
- added R47: 300, Resistor_SMD:R_0603_1608Metric, F.Cu at (82.9, 109.3)
- added R48: 300, Resistor_SMD:R_0603_1608Metric, F.Cu at (89.6, 109.3)
- added R49: 300, Resistor_SMD:R_0603_1608Metric, F.Cu at (103.8, 108.4)
- added R5: 4.7k, Resistor_SMD:R_0603_1608Metric, B.Cu at (128.5, 122.8)
- added R53: 10k, Resistor_SMD:R_0603_1608Metric, F.Cu at (86.0, 94.0)
- added R55: 10k, Resistor_SMD:R_0603_1608Metric, B.Cu at (82.5, 100.0)
- added R56: 10k, Resistor_SMD:R_0603_1608Metric, B.Cu at (98.1, 92.2)
- added R60: 10k, Resistor_SMD:R_0603_1608Metric, B.Cu at (89.8, 102.5)
- added R61: 10k, Resistor_SMD:R_0603_1608Metric, F.Cu at (103.0, 95.2)
- added R62: 10k, Resistor_SMD:R_0603_1608Metric, B.Cu at (100.7, 87.1)
- added R7: 5.1k, Resistor_SMD:R_0603_1608Metric, B.Cu at (122.4, 81.5)
- added R70: 22, Resistor_SMD:R_0603_1608Metric, F.Cu at (99.0, 101.8)
- added R71: 22, Resistor_SMD:R_0603_1608Metric, F.Cu at (88.5, 99.2)
- added R73: 22, Resistor_SMD:R_0603_1608Metric, F.Cu at (99.6, 92.2)
- added R74: 22, Resistor_SMD:R_0603_1608Metric, F.Cu at (101.5, 106.2)
- added R75: 10k, Resistor_SMD:R_0603_1608Metric, F.Cu at (98.2, 67.5)
- added R76: 53k6, Resistor_SMD:R_0603_1608Metric, F.Cu at (109.9, 96.7)
- added R77: 10k, Resistor_SMD:R_0603_1608Metric, B.Cu at (110.2, 65.7)
- added R78: 200k, Resistor_SMD:R_0603_1608Metric, F.Cu at (111.2, 103.2)
- added R79: 44.2k, Resistor_SMD:R_0603_1608Metric, F.Cu at (111.2, 101.8)
- added R8: 5.1k, Resistor_SMD:R_0603_1608Metric, B.Cu at (122.5, 84.4)
- added R80: 22, Resistor_SMD:R_0603_1608Metric, F.Cu at (100.7, 88.6)
- added R81: 10k, Resistor_SMD:R_0603_1608Metric, F.Cu at (91.6, 114.0)
- added R85: 10k, Resistor_SMD:R_0603_1608Metric, F.Cu at (98.6, 113.8)
- added R86: 10k, Resistor_SMD:R_0603_1608Metric, F.Cu at (84.4, 114.1)
- added R87: 10k, Resistor_SMD:R_0603_1608Metric, F.Cu at (77.3, 114.2)
- added R88: 10k, Resistor_SMD:R_0603_1608Metric, F.Cu at (80.6, 109.0)
- added R89: 10k, Resistor_SMD:R_0603_1608Metric, F.Cu at (87.3, 109.0)
- added R9: 220, Resistor_SMD:R_0603_1608Metric, F.Cu at (61.5, 72.2)
- added R90: 10k, Resistor_SMD:R_0603_1608Metric, F.Cu at (101.5, 108.6)
- added R91: 10k, Resistor_SMD:R_0603_1608Metric, F.Cu at (94.5, 108.8)
- added R92: 10k, Resistor_SMD:R_0603_1608Metric, F.Cu at (106.3, 91.5)
- added R93: 10k, Resistor_SMD:R_0603_1608Metric, F.Cu at (106.3, 88.4)
- added R94: 10k, Resistor_SMD:R_0603_1608Metric, F.Cu at (106.3, 85.4)
- added R95: 10k, Resistor_SMD:R_0603_1608Metric, F.Cu at (109.9, 98.2)
- added R96: 10k, Resistor_SMD:R_0603_1608Metric, B.Cu at (111.7, 65.7)
- added R97: 10k, Resistor_SMD:R_0603_1608Metric, B.Cu at (105.0, 65.6)
- added R98: 10k, Resistor_SMD:R_0603_1608Metric, B.Cu at (113.2, 65.7)
- added R99: 10k, Resistor_SMD:R_0603_1608Metric, B.Cu at (106.6, 65.6)
- added Rs1: 5m, Resistor_SMD:R_1206_3216Metric, F.Cu at (110.5, 105.2)
- added SW1: SW_Push, Button_Switch_SMD:SW_SPST_PTS810, F.Cu at (82.4, 94.0)
- added SW2: SW_SPDT, Button_Switch_SMD:SW_SPDT_CK_JS102011SAQN, F.Cu at (96.7, 62.1)
- added TP1: TestPoint, Burocket Logo:Burocket Logo, B.Cu at (65.1, 102.6)
- added U1: STM32F405RGT6, Package_QFP:LQFP-64_10x10mm_P0.5mm, F.Cu at (91.8, 86.4)
- added U10: INA226, Package_SO:TSSOP-10_3x3mm_P0.5mm, B.Cu at (130.2, 116.2)
- added U11: W25Q128JVS, Package_SO:SOIC-8_5.3x5.3mm_P1.27mm, F.Cu at (104.7, 100.7)
- added U12: TPS7A4701, Package_DFN_QFN:Texas_RGW0020A_VQFN-20-1EP_5x5mm_P0.65mm_EP3.15x3.15mm, F.Cu at (107.0, 80.0)
- added U14: TPS62933, Package_TO_SOT_SMD:SOT-583-8, F.Cu at (113.1, 99.6)
- added U4: TPD2EUSB30DRTR, Package_TO_SOT_SMD:Texas_DRT-3, F.Cu at (116.0, 83.1)
- added U5: MS5611, MS5611:SON8_MS5611_TEC, F.Cu at (87.8, 102.8)
- added U6: ICM-42688-P, ICM_42688_P:LGA14_2P5X3X0P91_TDK, F.Cu at (82.9, 100.1)
- added U7: ADXL375, ADXL375BCCZ_RL7:LGA_CC-14-1_ADI-L, F.Cu at (96.2, 101.9)
- added U8: TPS2121RUXR, footprints.ugly:RUX0012A, F.Cu at (116.4, 90.8)
- added U9: MAX-M10N, RF_GPS:ublox_MAX, F.Cu at (81.7, 73.2)
- added Y2: 25MHz, Crystal:Crystal_SMD_2520-4Pin_2.5x2.0mm, F.Cu at (82.7, 84.9)
Other:
- board text added: "X"
- board text added: "Y"
- board text added: "Z"
