File: Hardware/.history_trim/Power.kicad_sch (KiCad schematic)
At the start: 9 parts, among them J1 USB4105-GF-A-120, U4 TPD2EUSB30DRTR

Commit message: Purged heavy binaries and updated gitignore
Parts:
- removed C22: 100nF, Capacitor_SMD:C_0603_1608Metric, symbol Device:C
- removed C52: 22uF, Capacitor_SMD:C_0805_2012Metric, symbol Device:C
- removed D3: ESD321DYAR, Diode_SMD:D_SOD-523, symbol Diode:ESD5Zxx
- removed D4: Green LED, LED_SMD:LED_0603_1608Metric, symbol Device:LED
- removed J1: USB4105-GF-A-120, USB4105-GF-A-120:GCT_USB4105-GF-A-120, symbol USB4105-GF-A-120:USB4105-GF-A-120
- removed R15: 1k, Resistor_SMD:R_0603_1608Metric, symbol Device:R
- removed R7, R8: 5.1k, Resistor_SMD:R_0603_1608Metric, symbol Device:R
- removed U4: TPD2EUSB30DRTR, Package_TO_SOT_SMD:Texas_DRT-3, symbol Power_Protection:TPD2EUSB30A
- added BT1: Battery, Connector_AMASS:AMASS_XT60-F_1x02_P7.20mm_Vertical, symbol Device:Battery
- added C19, C20, C25, C26, C9: C, symbol Device:C
- added C23: 100nF, Capacitor_SMD:C_0402_1005Metric, symbol Device:C
- added C24: 0.1nF, Capacitor_SMD:C_0402_1005Metric, symbol Device:C
- added L1: 9.1uH, Inductor_SMD_Wurth:L_Wurth_WE-PDF-1045, symbol Device:L
- added R21: 100k, Resistor_SMD:R_0402_1005Metric, symbol Device:R
- added R22: 13.7K, Resistor_SMD:R_0402_1005Metric, symbol Device:R
- added R23: 412k, Resistor_SMD:R_0402_1005Metric, symbol Device:R
- added R24: 97.6K, Resistor_SMD:R_0402_1005Metric, symbol Device:R
- added U2: TPS54302, TPS54302DDCR:SOT95P280X110-6N, symbol TPS54302DDCR:TPS54302DDCR
- added U8: TPS2121RUXR, footprints.ugly:RUX0012A, symbol 2026-06-29_10-29-30:TPS2121RUXR
Connections:
- net GND: now also BT1.2 (-), C19.2, C20.2, C25.2, C26.2, C9.2, R22.2, R24.2, U2.1 (GND), U8.12 (GND)
- net VBUS: now also U8.2 (IN2)
- new net: C24.2, R21.2, R22.1, U2.4 (FB)
- new net: C23.1, U2.6 (BOOT)
- new net: C23.2, C24.1, L1.1, U2.2 (SW)
- new net: R23.2, R24.1, U2.5 (EN)
- new net: U8.1 (OUT), U8.8 (OUT)
- new net +5V: C25.1, C26.1, L1.2, R21.1, U8.7 (IN1)
- new net +BATT: BT1.1 (+), C19.1, C20.1, C9.1, R23.1, U2.3 (VIN)
- no-connect marks 2 -> 0
Other:
- note added: "----->"
- note added: "---->"
- note added: "2S BAT 6-8.4V"
- note added: "3.3V"
- note added: "5V"
- note added: "Buck converter"
- note added: "LDO"
- note added: "Power MUX"
- note added: "Power input ---->"
- note added: "TODO: Select input and output caps"
- note added: "USB-c ------>"
- note added: "UVLO = 6V"
- note added: "[2] Power"
- note removed: "USB-c Connector"
- note removed: "[5] USB-c"
- title: (none) -> Power
